File: hw-design/top-board/actuators.sch (KiCad schematic (older format))
At the start: 20 parts, among them P7 FOOTSWITCH, P8 FOOTSWITCH

Commit message: Changed SODIM to Marsboard header + added liniar regulator for audio codec
Parts:
- C39, C40, C41, C42: symbol C -> top-board-rescue:C
- E1, E2: symbol PEC11R -> local-components:PEC11R
- P7, P8: symbol CONN_01X02 -> top-board-rescue:CONN_01X02
- R15, R16, R17, R18, R19, R20, R21, R22, R23, R24, R25, R26: symbol R -> top-board-rescue:R
Changed lines of the file:
@@
-EESchema Schematic File Version 2
-LIBS:power
-LIBS:device
-LIBS:conn
-LIBS:regul
-LIBS:74xgxx
-LIBS:local-components
+EESchema Schematic File Version 4
 LIBS:top-board-cache
-EELAYER 25 0
+EELAYER 26 0
 EELAYER END
 $Descr A4 11693 8268
@@
 $EndDescr
 $Comp
-L CONN_01X02 P7
+L top-board-rescue:CONN_01X02 P7
 U 1 1 555278EA
 P 2100 2500
@@
 $EndComp
 $Comp
-L GNDD #PWR062
+L top-board-rescue:GNDD #PWR062
 U 1 1 555279A3
 P 2450 2650
@@
 $EndComp
 $Comp
-L R R15
+L top-board-rescue:R R15
 U 1 1 555279BF
 P 2450 2200
@@
 $EndComp
 $Comp
-L +3.3V #PWR063
+L top-board-rescue:+3.3V #PWR063
 U 1 1 55527A56
 P 2450 1950
@@
 $EndComp
 $Comp
-L CONN_01X02 P8
+L top-board-rescue:CONN_01X02 P8
 U 1 1 55527C76
 P 2100 3800
@@
 $EndComp
 $Comp
-L GNDD #PWR064
+L top-board-rescue:GNDD #PWR064
 U 1 1 55527C7C
 P 2450 3950
@@
 $EndComp
 $Comp
-L R R16
+L top-board-rescue:R R16
 U 1 1 55527C84
 P 2450 3500
@@
 $EndComp
 $Comp
-L +3.3V #PWR065
+L top-board-rescue:+3.3V #PWR065
 U 1 1 55527C8C
 P 2450 3250
@@
 $EndComp
 $Comp
-L PEC11R E1
+L local-components:PEC11R E1
 U 1 1 555621D2
 P 5100 2850
@@
 $EndComp
 $Comp
-L GNDD #PWR066
+L top-board-rescue:GNDD #PWR066
 U 1 1 55562530
 P 4700 2650
@@
 $EndComp
 $Comp
-L R R17
+L top-board-rescue:R R17
 U 1 1 555627D4
 P 5350 2200
@@
 $EndComp
 $Comp
-L +3.3V #PWR067
+L top-board-rescue:+3.3V #PWR067
 U 1 1 555627DC
 P 5350 1950
@@
 $EndComp
 $Comp
-L R R18
+L top-board-rescue:R R18
 U 1 1 55562ED4
 P 5600 2950
@@
 $EndComp
 $Comp
-L R R20
+L top-board-rescue:R R20
 U 1 1 5556305B
 P 5850 3200
@@
 $EndComp
 $Comp
-L GNDD #PWR068
+L top-board-rescue:GNDD #PWR068
 U 1 1 5556323B
 P 5100 3250
@@
 $EndComp
 $Comp
-L +3.3V #PWR069
+L top-board-rescue:+3.3V #PWR069
 U 1 1 55563E1D
 P 5600 2750
@@
 $EndComp
 $Comp
-L C C39
+L top-board-rescue:C C39
 U 1 1 555643DB
 P 6150 3450
@@
 $EndComp
 $Comp
-L GNDD #PWR070
+L top-board-rescue:GNDD #PWR070
 U 1 1 55564410
 P 6150 3700
@@
 $EndComp
 $Comp
-L R R19
+L top-board-rescue:R R19
 U 1 1 555654C6
 P 5600 3800
@@
 $EndComp
 $Comp
-L R R21
+L top-board-rescue:R R21
 U 1 1 555654CC
 P 5850 4050
@@
 $EndComp
 $Comp
-L +3.3V #PWR071
+L top-board-rescue:+3.3V #PWR071
 U 1 1 555654D6
 P 5600 3600
@@
 $EndComp
 $Comp
-L C C40
+L top-board-rescue:C C40
 U 1 1 555654DD
 P 6150 4300
@@
 $EndComp
 $Comp
-L GNDD #PWR072
+L top-board-rescue:GNDD #PWR072
 U 1 1 555654E3
 P 6150 4550
@@
 $EndComp
 $Comp
-L PEC11R E2
+L local-components:PEC11R E2
 U 1 1 55566FA7
 P 7300 2850
@@
 $EndComp
 $Comp
-L GNDD #PWR073
+L top-board-rescue:GNDD #PWR073
 U 1 1 55566FAD
 P 6900 2650
@@
 $EndComp
 $Comp
-L R R22
+L top-board-rescue:R R22
 U 1 1 55566FB6
 P 7550 2200
@@
 $EndComp
 $Comp
-L +3.3V #PWR074
+L top-board-rescue:+3.3V #PWR074
 U 1 1 55566FBF
 P 7550 1950
@@
 $EndComp
 $Comp
-L R R23
+L top-board-rescue:R R23
 U 1 1 55566FC9
 P 7800 2950
@@
 $EndComp
 $Comp
-L R R25
+L top-board-rescue:R R25
 U 1 1 55566FCF
 P 8050 3200
@@
 $EndComp
 $Comp
-L GNDD #PWR075
+L top-board-rescue:GNDD #PWR075
 U 1 1 55566FD5
 P 7300 3250
@@
 $EndComp
 $Comp
-L +3.3V #PWR076
+L top-board-rescue:+3.3V #PWR076
 U 1 1 55566FE3
 P 7800 2750
@@
 $EndComp
 $Comp
-L C C41
+L top-board-rescue:C C41
 U 1 1 55566FEA
 P 8350 3450
@@
 $EndComp
 $Comp
-L GNDD #PWR077
+L top-board-rescue:GNDD #PWR077
 U 1 1 55566FF0
 P 8350 3700
@@
 $EndComp
 $Comp
-L R R24
+L top-board-rescue:R R24
 U 1 1 55566FFA
 P 7800 3800
@@
 $EndComp
 $Comp
-L R R26
+L top-board-rescue:R R26
 U 1 1 55567000
 P 8050 4050
@@
 $EndComp
 $Comp
-L +3.3V #PWR078
+L top-board-rescue:+3.3V #PWR078
 U 1 1 5556700C
 P 7800 3600
@@
 $EndComp
 $Comp
-L C C42
+L top-board-rescue:C C42
 U 1 1 55567013
 P 8350 4300
@@
 $EndComp
 $Comp
-L GNDD #PWR079
+L top-board-rescue:GNDD #PWR079
 U 1 1 55567019
 P 8350 4550

Commit message: added logo's and updated gerber files
Parts:
- E1, E2: symbol local-components:PEC11R -> top-board-rescue:PEC11R-local-components
Changed lines of the file:
@@
 $EndComp
 $Comp
-L local-components:PEC11R E1
+L top-board-rescue:PEC11R-local-components E1
 U 1 1 555621D2
 P 5100 2850
@@
 $EndComp
 $Comp
-L local-components:PEC11R E2
+L top-board-rescue:PEC11R-local-components E2
 U 1 1 55566FA7
 P 7300 2850
