File: hw-design/top-board/cpu.sch (KiCad schematic (older format))
At the start: 35 parts, among them P2 ISP, P4 BOTTOM_CONN, Q1 2N7002, SW1 BT_RESET, U3 MCP6001, U4 LPC1759FBD80, Y1 10MHz

Commit message: Changed SODIM to Marsboard header + added liniar regulator for audio codec
Parts:
- C10, C11, C12, C13, C14, C15, C16, C5, C6, C7, C8, C9: symbol C -> top-board-rescue:C
- D1, D2, D3: symbol D -> top-board-rescue:D
- P2: symbol CONN_02X05 -> top-board-rescue:CONN_02X05
- P4: symbol CONN_02X10 -> top-board-rescue:CONN_02X10
- Q1: symbol Q_NMOS_GSD -> top-board-rescue:Q_NMOS_GSD
- R1, R10, R11, R12, R2, R3, R4, R5, R6, R7, R8, R9: symbol R -> top-board-rescue:R
- RP1: symbol R_PACK4 -> top-board-rescue:R_PACK4
- SW1: symbol SW_PUSH -> top-board-rescue:SW_PUSH
- U3: symbol MCP6001 -> local-components:MCP6001
- U4: symbol LPC1759FBD80 -> local-components:LPC1759FBD80
- Y1: symbol Crystal_Small -> top-board-rescue:Crystal_Small
Changed lines of the file:
@@
-EESchema Schematic File Version 2
-LIBS:power
-LIBS:device
-LIBS:conn
-LIBS:regul
-LIBS:74xgxx
-LIBS:local-components
+EESchema Schematic File Version 4
 LIBS:top-board-cache
-EELAYER 25 0
+EELAYER 26 0
 EELAYER END
 $Descr A4 11693 8268
@@
 $EndDescr
 $Comp
-L LPC1759FBD80 U4
+L local-components:LPC1759FBD80 U4
 U 1 1 55528434
 P 7250 3950
@@
 $EndComp
 $Comp
-L GNDD #PWR014
+L top-board-rescue:GNDD #PWR014
 U 1 1 555285E7
 P 6750 6300
@@
 $EndComp
 $Comp
-L GNDD #PWR015
+L top-board-rescue:GNDD #PWR015
 U 1 1 55528602
 P 7550 6300
@@
 $EndComp
 $Comp
-L +3.3V #PWR016
+L top-board-rescue:+3.3V #PWR016
 U 1 1 55528786
 P 9050 5600
@@
 $EndComp
 $Comp
-L C C16
+L top-board-rescue:C C16
 U 1 1 5552879E
 P 9050 5850
@@
 $EndComp
 $Comp
-L GNDD #PWR017
+L top-board-rescue:GNDD #PWR017
 U 1 1 5552888B
 P 8900 6100
@@
 $EndComp
 $Comp
-L C C9
+L top-board-rescue:C C9
 U 1 1 555289F5
 P 5600 1200
@@
 $EndComp
 $Comp
-L C C10
+L top-board-rescue:C C10
 U 1 1 55528C0F
 P 5900 1200
@@
 $EndComp
 $Comp
-L C C11
+L top-board-rescue:C C11
 U 1 1 55528C35
 P 6200 1200
@@
 $EndComp
 $Comp
-L C C12
+L top-board-rescue:C C12
 U 1 1 55528CCE
 P 6500 1200
@@
 $EndComp
 $Comp
-L C C15
+L top-board-rescue:C C15
 U 1 1 55528CF2
 P 8650 1200
@@
 $EndComp
 $Comp
-L C C14
+L top-board-rescue:C C14
 U 1 1 55528D80
 P 8350 1200
@@
 $EndComp
 $Comp
-L C C13
+L top-board-rescue:C C13
 U 1 1 55528DA8
 P 8050 1200
@@
 $EndComp
 $Comp
-L GNDD #PWR018
+L top-board-rescue:GNDD #PWR018
 U 1 1 55528F85
 P 6500 1550
@@
 $EndComp
 $Comp
-L +3.3V #PWR019
+L top-board-rescue:+3.3V #PWR019
 U 1 1 555294F0
 P 6500 800
@@
 $EndComp
 $Comp
-L +3.3V #PWR020
+L top-board-rescue:+3.3V #PWR020
 U 1 1 5552A974
 P 8650 800
@@
 $EndComp
 $Comp
-L GNDD #PWR021
+L top-board-rescue:GNDD #PWR021
 U 1 1 5552AA32
 P 8650 1550
@@
 $EndComp
 $Comp
-L +3.3V #PWR022
+L top-board-rescue:+3.3V #PWR022
 U 1 1 5552AC13
 P 6850 1550
@@
 $EndComp
 $Comp
-L +3.3V #PWR023
+L top-board-rescue:+3.3V #PWR023
 U 1 1 5552AD6D
 P 7350 1550
@@
 $EndComp
 $Comp
-L +3.3V #PWR024
+L top-board-rescue:+3.3V #PWR024
 U 1 1 5552AE14
 P 7650 1550
@@
 $EndComp
 $Comp
-L +3.3V #PWR025
+L top-board-rescue:+3.3V #PWR025
 U 1 1 5552B0DD
 P 5500 5600
@@
 $EndComp
 $Comp
-L Crystal_Small Y1
+L top-board-rescue:Crystal_Small Y1
 U 1 1 5552B69D
 P 5400 5100
@@
 $EndComp
 $Comp
-L C C7
+L top-board-rescue:C C7
 U 1 1 5552BBA9
 P 4850 5450
@@
 $EndComp
 $Comp
-L C C8
+L top-board-rescue:C C8
 U 1 1 5552BC14
 P 5150 5450
@@
 $EndComp
 $Comp
-L GNDD #PWR026
+L top-board-rescue:GNDD #PWR026
 U 1 1 5552C790
 P 4850 5700
@@
 $EndComp
 $Comp
-L GNDD #PWR027
+L top-board-rescue:GNDD #PWR027
 U 1 1 5552C840
 P 5150 5700
@@
 $EndComp
 $Comp
-L CONN_02X10 P4
+L top-board-rescue:CONN_02X10 P4
 U 1 1 5555C389
 P 2750 4250
@@
 $EndComp
 $Comp
-L R R12
+L top-board-rescue:R R12
 U 1 1 55569C10
 P 9950 4900
@@
 $EndComp
 $Comp
-L +3.3V #PWR028
+L top-board-rescue:+3.3V #PWR028
 U 1 1 55569FE3
 P 9950 4650
@@
 $EndComp
 $Comp
-L CONN_02X05 P2
+L top-board-rescue:CONN_02X05 P2
 U 1 1 5556D1BD
 P 1700 6350
@@
 $EndComp
 $Comp
-L GNDD #PWR029
+L top-board-rescue:GNDD #PWR029
 U 1 1 5556D3DF
 P 1350 6650
@@
 $EndComp
 $Comp
-L R R5
+L top-board-rescue:R R5
 U 1 1 5556D746
 P 2050 5900
@@
 $EndComp
 $Comp
-L R R7
+L top-board-rescue:R R7
 U 1 1 5556DB27
 P 2150 5900
@@
 $EndComp
 $Comp
-L R R10
+L top-board-rescue:R R10
 U 1 1 5556DB65
 P 2400 5900
@@
 $EndComp
 $Comp
-L R R8
+L top-board-rescue:R R8
 U 1 1 5556DB9D
 P 2250 5900
@@
 $EndComp
 $Comp
-L +3.3V #PWR030
+L top-board-rescue:+3.3V #PWR030
 U 1 1 5556E77E
 P 2050 5500
@@
 $EndComp
 $Comp
-L GNDD #PWR031
+L top-board-rescue:GNDD #PWR031
 U 1 1 5557BBA5
 P 3100 4800
@@
 $EndComp
 $Comp
-L GNDD #PWR032
+L top-board-rescue:GNDD #PWR032
 U 1 1 5557C69D
 P 2400 4800
@@
 $EndComp
 $Comp
-L SW_PUSH SW1
+L top-board-rescue:SW_PUSH SW1
 U 1 1 555AC0FD
 P 3900 1950
@@
 NoConn ~ 8850 2050
 $Comp
-L R R4
+L top-board-rescue:R R4
 U 1 1 55F055B6
 P 2000 3550
@@
 $EndComp
 $Comp
-L R R6
+L top-board-rescue:R R6
 U 1 1 55F06095
 P 2150 3550
@@
 $EndComp
 $Comp
-L +3.3V #PWR033
+L top-board-rescue:+3.3V #PWR033
 U 1 1 55F07936
 P 2150 3200
@@
 $EndComp
 $Comp
-L R R9
+L top-board-rescue:R R9
 U 1 1 55F0813F
 P 2300 3550
@@
 $EndComp
 $Comp
-L MCP6001 U3
+L local-components:MCP6001 U3
 U 1 1 55F0ECA7
 P 2750 1550
@@
 $EndComp
 $Comp
-L R R2
+L top-board-rescue:R R2
 U 1 1 55F0F70F
 P 1950 1200
@@
 $EndComp
 $Comp
-L R R3
+L top-board-rescue:R R3
 U 1 1 55F0FE88
 P 1950 1300
@@
 $EndComp
 $Comp
-L +3.3V #PWR034
+L top-board-rescue:+3.3V #PWR034
 U 1 1 55F1048B
 P 1650 1150
@@
 $EndComp
 $Comp
-L D D1
+L top-board-rescue:D D1
 U 1 1 55F10910
 P 1850 1800
@@
 $EndComp
 $Comp
-L R R1
+L top-board-rescue:R R1
 U 1 1 55F10ABB
 P 1850 1650
@@
 $EndComp
 $Comp
-L C C5
+L top-board-rescue:C C5
 U 1 1 55F117E5
 P 2250 2000
@@
 $EndComp
 $Comp
-L GNDD #PWR035
+L top-board-rescue:GNDD #PWR035
 U 1 1 55F12F83
 P 2650 1950
@@
 $EndComp
 $Comp
-L GNDD #PWR036
+L top-board-rescue:GNDD #PWR036
 U 1 1 55F1337A
 P 1650 1350
@@
 $EndComp
 $Comp
-L GNDD #PWR037
+L top-board-rescue:GNDD #PWR037
 U 1 1 55F133A2
 P 2250 2250
@@
 $EndComp
 $Comp
-L +3.3V #PWR038
+L top-board-rescue:+3.3V #PWR038
 U 1 1 55F14423
 P 2650 1150
@@
 HMI_RESET
 $Comp
-L C C6
+L top-board-rescue:C C6
 U 1 1 55F21E4D
 P 3600 1900
@@
 Connection ~ 3600 1550
 $Comp
-L GNDD #PWR039
+L top-board-rescue:GNDD #PWR039
 U 1 1 55F257D4
 P 3600 2150
@@
 	3600 2050 3600 2150
 $Comp
-L +3.3V #PWR040
+L top-board-rescue:+3.3V #PWR040
 U 1 1 55F263E7
 P 3600 950
@@
 	3600 950  3600 1050
 $Comp
-L D D3
+L top-board-rescue:D D3
 U 1 1 55F2AF8C
 P 3350 1550
@@
 	3500 1550 4100 1550
 $Comp
-L GNDD #PWR041
+L top-board-rescue:GNDD #PWR041
 U 1 1 55F2C2DC
 P 3900 2300
@@
 JTAG_RESET
 $Comp
-L D D2
+L top-board-rescue:D D2
 U 1 1 55F31488
 P 2250 6550
@@
 	5500 3850 5650 3850
 $Comp
-L Q_NMOS_GSD Q1
+L top-board-rescue:Q_NMOS_GSD Q1
 U 1 1 55F4008F
 P 10050 5450
@@
 Connection ~ 9950 5150
 $Comp
-L GNDD #PWR042
+L top-board-rescue:GNDD #PWR042
 U 1 1 55F415F1
 P 9950 5800
@@
 	1950 6350 2600 6350
 $Comp
-L GNDD #PWR043
+L top-board-rescue:GNDD #PWR043
 U 1 1 55F44C3F
 P 2700 5750
@@
 Connection ~ 2400 6350
 $Comp
-L R R11
+L top-board-rescue:R R11
 U 1 1 55F47A93
 P 3600 1200
@@
 $EndComp
 $Comp
-L R_PACK4 RP1
+L top-board-rescue:R_PACK4 RP1
 U 1 1 55F2C432
 P 2100 7350

Commit message: added logo's and updated gerber files
Parts:
- U3: symbol local-components:MCP6001 -> top-board-rescue:MCP6001-local-components
- U4: symbol local-components:LPC1759FBD80 -> top-board-rescue:LPC1759FBD80-local-components
Changed lines of the file:
@@
 $EndDescr
 $Comp
-L local-components:LPC1759FBD80 U4
+L top-board-rescue:LPC1759FBD80-local-components U4
 U 1 1 55528434
 P 7250 3950
@@
 $EndComp
 $Comp
-L local-components:MCP6001 U3
+L top-board-rescue:MCP6001-local-components U3
 U 1 1 55F0ECA7
 P 2750 1550
@@
 	7550 6150 7550 6300
 Wire Wire Line
-	6750 6150 6750 6300
-Wire Wire Line
-	6750 6250 7250 6250
+	6750 6150 6750 6250
+Wire Wire Line
+	6750 6250 6850 6250
 Wire Wire Line
 	7250 6250 7250 6150
@@
 	8850 5850 8900 5850
 Wire Wire Line
-	8900 5850 8900 6100
-Wire Wire Line
-	9050 5600 9050 5700
+	8900 5850 8900 6050
+Wire Wire Line
+	9050 5600 9050 5650
 Wire Wire Line
 	8850 5650 9050 5650
@@
 	5600 1050 5600 900
 Wire Wire Line
-	6500 1350 6500 1550
-Wire Wire Line
-	5600 1450 6500 1450
+	6500 1350 6500 1450
+Wire Wire Line
+	5600 1450 5900 1450
 Wire Wire Line
 	5900 1050 5900 900
@@
 	6200 900  6200 1050
 Wire Wire Line
-	6500 800  6500 1050
+	6500 800  6500 900
 Wire Wire Line
 	5900 1350 5900 1450
@@
 	6200 1350 6200 1450
 Wire Wire Line
-	5600 900  6500 900
+	5600 900  5900 900
 Wire Wire Line
 	5600 1450 5600 1350
 Wire Wire Line
-	8650 800  8650 1050
+	8650 800  8650 900
 Wire Wire Line
 	8050 1050 8050 900
 Wire Wire Line
-	8050 900  8650 900
+	8050 900  8350 900
 Wire Wire Line
 	8350 1050 8350 900
 Wire Wire Line
-	8650 1350 8650 1550
+	8650 1350 8650 1450
 Wire Wire Line
 	8050 1350 8050 1450
 Wire Wire Line
-	8050 1450 8650 1450
+	8050 1450 8350 1450
 Wire Wire Line
 	8350 1350 8350 1450
 Wire Wire Line
-	6850 1550 6850 1750
+	6850 1550 6850 1650
 Wire Wire Line
 	7150 1650 7150 1750
 Wire Wire Line
-	6850 1650 7150 1650
+	6850 1650 6950 1650
 Wire Wire Line
 	6950 1750 6950 1650
@@
 	7050 1750 7050 1650
 Wire Wire Line
-	7350 1550 7350 1750
+	7350 1550 7350 1650
 Wire Wire Line
 	7450 1750 7450 1650
@@
 	5600 5050 5600 4950
 Wire Wire Line
-	5600 4950 4850 4950
+	5600 4950 5400 4950
 Wire Wire Line
 	4850 4950 4850 5300
@@
 	5600 5150 5600 5250
 Wire Wire Line
-	5600 5250 5150 5250
+	5600 5250 5400 5250
 Wire Wire Line
 	5150 5250 5150 5300
@@
 	9000 4650 8850 4650
 Wire Wire Line
-	1850 4600 2500 4600
-Wire Wire Line
-	1850 4700 2500 4700
+	1850 4600 2150 4600
+Wire Wire Line
+	1850 4700 2000 4700
 Wire Wire Line
 	5650 3250 5500 3250
@@
 	1450 6250 1350 6250
 Wire Wire Line
-	1350 6250 1350 6650
+	1350 6250 1350 6350
 Wire Wire Line
 	1450 6350 1350 6350
@@
 	1450 6550 1350 6550
 Wire Wire Line
-	1950 6150 2600 6150
-Wire Wire Line
-	1950 6250 2600 6250
-Wire Wire Line
-	1950 6450 2600 6450
+	1950 6150 2050 6150
+Wire Wire Line
+	1950 6250 2150 6250
+Wire Wire Line
+	1950 6450 2250 6450
 Wire Wire Line
 	2050 6050 2050 6150
@@
 	2250 6050 2250 6450
 Wire Wire Line
-	2050 5500 2050 5750
+	2050 5500 2050 5600
 Wire Wire Line
 	2250 5600 2250 5750
@@
 	1850 4400 2500 4400
 Wire Wire Line
-	1850 4500 2500 4500
+	1850 4500 2300 4500
 Wire Wire Line
 	3000 3900 3300 3900
@@
 	3000 3800 3100 3800
 Wire Wire Line
-	3100 3800 3100 4800
+	3100 3800 3100 4300
 Wire Wire Line
 	3000 4300 3100 4300
@@
 	2500 4000 2400 4000
 Wire Wire Line
-	2400 4000 2400 4800
+	2400 4000 2400 4300
 Wire Wire Line
 	2500 4300 2400 4300
@@
 	1000 2650 1000 5050
 Wire Wire Line
-	5400 2750 5650 2750
+	5400 2750 5550 2750
 Wire Notes Line
 	1000 2550 4450 2550
@@
 	9950 4750 9950 4650
 Wire Wire Line
-	2150 3200 2150 3400
+	2150 3200 2150 3300
 Wire Wire Line
 	2000 3400 2000 3300
 Wire Wire Line
-	2000 3300 2300 3300
+	2000 3300 2150 3300
 Connection ~ 2150 3300
 Wire Wire Line
@@
 Connection ~ 2000 4700
 Wire Wire Line
-	2050 5600 2250 5600
+	2050 5600 2150 5600
 Wire Wire Line
 	2100 6550 1950 6550
@@
 	1650 1300 1800 1300
 Wire Wire Line
-	2000 1650 2400 1650
+	2000 1650 2100 1650
 Wire Wire Line
 	2250 1850 2250 1650
 Connection ~ 2250 1650
 Wire Wire Line
-	1500 1650 1700 1650
-Wire Wire Line
-	3600 1350 3600 1750
+	1500 1650 1600 1650
+Wire Wire Line
+	3600 1350 3600 1550
 Wire Wire Line
 	1700 1800 1600 1800
@@
 	2100 1300 2250 1300
 Wire Wire Line
-	2250 1200 2250 1450
+	2250 1200 2250 1300
 Wire Wire Line
 	2250 1450 2400 1450
@@
 	3200 1550 3100 1550
 Wire Wire Line
-	3500 1550 4100 1550
+	3500 1550 3600 1550
 $Comp
 L top-board-rescue:GNDD #PWR041
@@
 $EndComp
 Wire Wire Line
-	9950 5050 9950 5250
+	9950 5050 9950 5150
 Wire Wire Line
 	8850 5150 9950 5150
@@
 	9950 5650 9950 5800
 Wire Wire Line
-	1950 6350 2600 6350
+	1950 6350 2400 6350
 $Comp
 L top-board-rescue:GNDD #PWR043
@@
 NoConn ~ 5650 4550
 NoConn ~ 5650 4650
+Wire Wire Line
+	6850 6250 6950 6250
+Wire Wire Line
+	6950 6250 7050 6250
+Wire Wire Line
+	7050 6250 7150 6250
+Wire Wire Line
+	7150 6250 7250 6250
+Wire Wire Line
+	6750 6250 6750 6300
+Wire Wire Line
+	9050 5650 9050 5700
+Wire Wire Line
+	8900 6050 8900 6100
+Wire Wire Line
+	5900 900  6200 900
+Wire Wire Line
+	6200 900  6500 900
+Wire Wire Line
+	6500 900  6500 1050
+Wire Wire Line
+	5900 1450 6200 1450
+Wire Wire Line
+	6200 1450 6500 1450
+Wire Wire Line
+	6500 1450 6500 1550
+Wire Wire Line
+	8650 900  8650 1050
+Wire Wire Line
+	8350 900  8650 900
+Wire Wire Line
+	8650 1450 8650 1550
+Wire Wire Line
+	8350 1450 8650 1450
+Wire Wire Line
+	6850 1650 6850 1750
+Wire Wire Line
+	6950 1650 7050 1650
+Wire Wire Line
+	7050 1650 7150 1650
+Wire Wire Line
+	7350 1650 7350 1750
+Wire Wire Line
+	5400 5250 5150 5250
+Wire Wire Line
+	5400 4950 4850 4950
+Wire Wire Line
+	1350 6350 1350 6550
+Wire Wire Line
+	1350 6550 1350 6650
+Wire Wire Line
+	2050 6150 2600 6150
+Wire Wire Line
+	2150 6250 2600 6250
+Wire Wire Line
+	2250 6450 2600 6450
+Wire Wire Line
+	2150 5600 2250 5600
+Wire Wire Line
+	2050 5600 2050 5750
+Wire Wire Line
+	3100 4300 3100 4800
+Wire Wire Line
+	2400 4300 2400 4800
+Wire Wire Line
+	2150 3300 2150 3400
+Wire Wire Line
+	2150 3300 2300 3300
+Wire Wire Line
+	2300 4500 2500 4500
+Wire Wire Line
+	2150 4600 2500 4600
+Wire Wire Line
+	2000 4700 2500 4700
+Wire Wire Line
+	2250 1650 2400 1650
+Wire Wire Line
+	1600 1650 1700 1650
+Wire Wire Line
+	2100 1650 2250 1650
+Wire Wire Line
+	2250 1300 2250 1450
+Wire Wire Line
+	3600 1550 3600 1750
+Wire Wire Line
+	3600 1550 3900 1550
+Wire Wire Line
+	3900 1550 4100 1550
+Wire Wire Line
+	5550 2750 5650 2750
+Wire Wire Line
+	9950 5150 9950 5250
+Wire Wire Line
+	2400 6350 2600 6350
 $EndSCHEMATC
