File: hw-design/top-board/display.sch (KiCad schematic (older format))
At the start: 32 parts, among them P5 BACKLIGHT, P6 BACKLIGHT, Q2 MMBT2222A, Q3 MMBT2222A

Commit message: Changed SODIM to Marsboard header + added liniar regulator for audio codec
Parts:
- C17, C18, C19, C20, C21, C22, C23, C24, C25, C26, C27, C28, C29, C30, C31, C32, C33, C34, C35, C36, C37, C38: symbol C -> top-board-rescue:C
- GLCD1, GLCD2: symbol ERC12864-2 -> local-components:ERC12864-2
- P5, P6: symbol CONN_01X02 -> top-board-rescue:CONN_01X02
- Q2, Q3: symbol Q_NPN_BEC -> top-board-rescue:Q_NPN_BEC
- R13, R14, R45, R46: symbol R -> top-board-rescue:R
Changed lines of the file:
@@
-EESchema Schematic File Version 2
-LIBS:power
-LIBS:device
-LIBS:conn
-LIBS:regul
-LIBS:74xgxx
-LIBS:local-components
+EESchema Schematic File Version 4
 LIBS:top-board-cache
-EELAYER 25 0
+EELAYER 26 0
 EELAYER END
 $Descr A4 11693 8268
@@
 $EndDescr
 $Comp
-L ERC12864-2 GLCD1
+L local-components:ERC12864-2 GLCD1
 U 1 1 55569CD0
 P 5200 1700
@@
 $EndComp
 $Comp
-L C C23
+L top-board-rescue:C C23
 U 1 1 5554C8A8
 P 3600 1900
@@
 $EndComp
 $Comp
-L C C22
+L top-board-rescue:C C22
 U 1 1 5554C9A0
 P 3600 1700
@@
 $EndComp
 $Comp
-L C C21
+L top-board-rescue:C C21
 U 1 1 5554CA08
 P 3600 1500
@@
 $EndComp
 $Comp
-L C C27
+L top-board-rescue:C C27
 U 1 1 5554D01D
 P 6600 2200
@@
 $EndComp
 $Comp
-L C C29
+L top-board-rescue:C C29
 U 1 1 5554D0CA
 P 6800 2100
@@
 $EndComp
 $Comp
-L C C31
+L top-board-rescue:C C31
 U 1 1 5554D12E
 P 7000 2000
@@
 $EndComp
 $Comp
-L C C33
+L top-board-rescue:C C33
 U 1 1 5554D717
 P 7200 1900
@@
 $EndComp
 $Comp
-L C C35
+L top-board-rescue:C C35
 U 1 1 5554D74B
 P 7400 1800
@@
 $EndComp
 $Comp
-L C C37
+L top-board-rescue:C C37
 U 1 1 5554D7DE
 P 7600 1700
@@
 $EndComp
 $Comp
-L GNDD #PWR044
+L top-board-rescue:GNDD #PWR044
 U 1 1 5554D90D
 P 6600 2550
@@
 $EndComp
 $Comp
-L GNDD #PWR045
+L top-board-rescue:GNDD #PWR045
 U 1 1 5554E711
 P 3800 2200
@@
 $EndComp
 $Comp
-L C C17
+L top-board-rescue:C C17
 U 1 1 5554EB42
 P 2750 1600
@@
 $EndComp
 $Comp
-L GNDD #PWR046
+L top-board-rescue:GNDD #PWR046
 U 1 1 5554EF2C
 P 2750 1950
@@
 $EndComp
 $Comp
-L +3.3V #PWR047
+L top-board-rescue:+3.3V #PWR047
 U 1 1 5554F071
 P 3800 1200
@@
 $EndComp
 $Comp
-L GNDD #PWR048
+L top-board-rescue:GNDD #PWR048
 U 1 1 5554F63A
 P 4500 2500
@@
 $EndComp
 $Comp
-L +3.3V #PWR049
+L top-board-rescue:+3.3V #PWR049
 U 1 1 55550113
 P 4150 2500
@@
 $EndComp
 $Comp
-L ERC12864-2 GLCD2
+L local-components:ERC12864-2 GLCD2
 U 1 1 5554DE46
 P 5200 4300
@@
 $EndComp
 $Comp
-L C C26
+L top-board-rescue:C C26
 U 1 1 5554DE4C
 P 3600 4500
@@
 $EndComp
 $Comp
-L C C25
+L top-board-rescue:C C25
 U 1 1 5554DE52
 P 3600 4300
@@
 $EndComp
 $Comp
-L C C24
+L top-board-rescue:C C24
 U 1 1 5554DE58
 P 3600 4100
@@
 $EndComp
 $Comp
-L C C28
+L top-board-rescue:C C28
 U 1 1 5554DE5F
 P 6600 4800
@@
 $EndComp
 $Comp
-L C C30
+L top-board-rescue:C C30
 U 1 1 5554DE65
 P 6800 4700
@@
 $EndComp
 $Comp
-L C C32
+L top-board-rescue:C C32
 U 1 1 5554DE6B
 P 7000 4600
@@
 $EndComp
 $Comp
-L C C34
+L top-board-rescue:C C34
 U 1 1 5554DE71
 P 7200 4500
@@
 $EndComp
 $Comp
-L C C36
+L top-board-rescue:C C36
 U 1 1 5554DE77
 P 7400 4400
@@
 $EndComp
 $Comp
-L C C38
+L top-board-rescue:C C38
 U 1 1 5554DE7D
 P 7600 4300
@@
 $EndComp
 $Comp
-L GNDD #PWR050
+L top-board-rescue:GNDD #PWR050
 U 1 1 5554DE83
 P 6600 5150
@@
 $EndComp
 $Comp
-L GNDD #PWR051
+L top-board-rescue:GNDD #PWR051
 U 1 1 5554DE89
 P 3800 4800
@@
 $EndComp
 $Comp
-L GNDD #PWR052
+L top-board-rescue:GNDD #PWR052
 U 1 1 5554DE9B
 P 2750 4550
@@
 $EndComp
 $Comp
-L +3.3V #PWR053
+L top-board-rescue:+3.3V #PWR053
 U 1 1 5554DEA1
 P 3800 3800
@@
 $EndComp
 $Comp
-L GNDD #PWR054
+L top-board-rescue:GNDD #PWR054
 U 1 1 5554DEA7
 P 4500 5100
@@
 $EndComp
 $Comp
-L +3.3V #PWR055
+L top-board-rescue:+3.3V #PWR055
 U 1 1 5554DEAD
 P 4150 5100
@@
 $EndComp
 $Comp
-L CONN_01X02 P5
+L top-board-rescue:CONN_01X02 P5
 U 1 1 555517B2
 P 9250 1400
@@
 $EndComp
 $Comp
-L GNDD #PWR056
+L top-board-rescue:GNDD #PWR056
 U 1 1 55554DEF
 P 9200 2350
@@
 $EndComp
 $Comp
-L R R13
+L top-board-rescue:R R13
 U 1 1 55556029
 P 8650 2050
@@
 $EndComp
 $Comp
-L CONN_01X02 P6
+L top-board-rescue:CONN_01X02 P6
 U 1 1 55557460
 P 9250 4000
@@
 $EndComp
 $Comp
-L GNDD #PWR057
+L top-board-rescue:GNDD #PWR057
 U 1 1 55557475
 P 9200 4950
@@
 $EndComp
 $Comp
-L R R14
+L top-board-rescue:R R14
 U 1 1 55557487
 P 8650 4650
@@
 $EndComp
 $Comp
-L Q_NPN_BEC Q2
+L top-board-rescue:Q_NPN_BEC Q2
 U 1 1 55559D02
 P 9100 2050
@@
 $EndComp
 $Comp
-L +3.3V #PWR058
+L top-board-rescue:+3.3V #PWR058
 U 1 1 555B6BEC
 P 5400 2800
@@
 $EndComp
 $Comp
-L C C19
+L top-board-rescue:C C19
 U 1 1 555B60DF
 P 3050 1600
@@
 $EndComp
 $Comp
-L C C20
+L top-board-rescue:C C20
 U 1 1 555B6F5D
 P 3050 4200
@@
 $EndComp
 $Comp
-L C C18
+L top-board-rescue:C C18
 U 1 1 555B837B
 P 2750 4200
@@
 	5400 2900 5600 2900
 $Comp
-L +3.3V #PWR059
+L top-board-rescue:+3.3V #PWR059
 U 1 1 55F4BD57
 P 5400 5400
@@
 	5400 5500 5600 5500
 $Comp
-L +12V #PWR060
+L top-board-rescue:+12V #PWR060
 U 1 1 5609A840
 P 9650 1300
@@
 $EndComp
 $Comp
-L R R45
+L top-board-rescue:R R45
 U 1 1 5609C39F
 P 9650 1500
@@
 	9650 1300 9650 1350
 $Comp
-L +12V #PWR061
+L top-board-rescue:+12V #PWR061
 U 1 1 5609DE0B
 P 9650 3900
@@
 $EndComp
 $Comp
-L R R46
+L top-board-rescue:R R46
 U 1 1 5609DE12
 P 9650 4100
@@
 	8800 2050 8900 2050
 $Comp
-L Q_NPN_BEC Q3
+L top-board-rescue:Q_NPN_BEC Q3
 U 1 1 561C2BD2
 P 9100 4650

Commit message: added logo's and updated gerber files
Parts:
- GLCD1, GLCD2: symbol local-components:ERC12864-2 -> top-board-rescue:ERC12864-2-local-components
Changed lines of the file:
@@
 $EndDescr
 $Comp
-L local-components:ERC12864-2 GLCD1
+L top-board-rescue:ERC12864-2-local-components GLCD1
 U 1 1 55569CD0
 P 5200 1700
@@
 $EndComp
 $Comp
-L local-components:ERC12864-2 GLCD2
+L top-board-rescue:ERC12864-2-local-components GLCD2
 U 1 1 5554DE46
 P 5200 4300
