File: hw-design/top-board/leds.sch (KiCad schematic (older format))
At the start: 26 parts, among them U5 PCA9685

Commit message: Changed SODIM to Marsboard header + added liniar regulator for audio codec
Parts:
- D4, D5, D6, D7, D8, D9: symbol LED_RGB -> top-board-rescue:LED_RGB
- R27, R28, R29, R30, R31, R32, R33, R34, R35, R36, R37, R38, R39, R40, R41, R42, R43, R44, R47: symbol R -> top-board-rescue:R
- U5: symbol PCA9685 -> local-components:PCA9685
Changed lines of the file:
@@
-EESchema Schematic File Version 2
-LIBS:power
-LIBS:device
-LIBS:conn
-LIBS:regul
-LIBS:74xgxx
-LIBS:local-components
+EESchema Schematic File Version 4
 LIBS:top-board-cache
-EELAYER 25 0
+EELAYER 26 0
 EELAYER END
 $Descr A4 11693 8268
@@
 $EndDescr
 $Comp
-L LED_RGB D4
+L top-board-rescue:LED_RGB D4
 U 1 1 5551D0C7
 P 2800 2050
@@
 $EndComp
 $Comp
-L R R27
+L top-board-rescue:R R27
 U 1 1 5551D2F4
 P 2250 1850
@@
 $EndComp
 $Comp
-L R R28
+L top-board-rescue:R R28
 U 1 1 5551D481
 P 2250 2050
@@
 $EndComp
 $Comp
-L R R29
+L top-board-rescue:R R29
 U 1 1 5551D4A1
 P 2250 2250
@@
 $EndComp
 $Comp
-L +3.3V #PWR080
+L top-board-rescue:+3.3V #PWR080
 U 1 1 5551D612
 P 3100 1700
@@
 $EndComp
 $Comp
-L LED_RGB D5
+L top-board-rescue:LED_RGB D5
 U 1 1 5551E569
 P 2800 3150
@@
 $EndComp
 $Comp
-L R R30
+L top-board-rescue:R R30
 U 1 1 5551E56F
 P 2250 2950
@@
 $EndComp
 $Comp
-L R R31
+L top-board-rescue:R R31
 U 1 1 5551E575
 P 2250 3150
@@
 $EndComp
 $Comp
-L R R32
+L top-board-rescue:R R32
 U 1 1 5551E57B
 P 2250 3350
@@
 $EndComp
 $Comp
-L +3.3V #PWR081
+L top-board-rescue:+3.3V #PWR081
 U 1 1 5551E584
 P 3100 2800
@@
 $EndComp
 $Comp
-L GNDD #PWR082
+L top-board-rescue:GNDD #PWR082
 U 1 1 5551E597
 P 9200 2350
@@
 $EndComp
 $Comp
-L R R44
+L top-board-rescue:R R44
 U 1 1 5552240D
 P 8350 5550
@@
 $EndComp
 $Comp
-L R R43
+L top-board-rescue:R R43
 U 1 1 55522407
 P 8350 5350
@@
 $EndComp
 $Comp
-L R R42
+L top-board-rescue:R R42
 U 1 1 55522401
 P 8350 5150
@@
 $EndComp
 $Comp
-L LED_RGB D9
+L top-board-rescue:LED_RGB D9
 U 1 1 555223FB
 P 8900 5350
@@
 $EndComp
 $Comp
-L R R41
+L top-board-rescue:R R41
 U 1 1 555223D1
 P 8350 4450
@@
 $EndComp
 $Comp
-L R R40
+L top-board-rescue:R R40
 U 1 1 555223CB
 P 8350 4250
@@
 $EndComp
 $Comp
-L R R39
+L top-board-rescue:R R39
 U 1 1 555223C5
 P 8350 4050
@@
 $EndComp
 $Comp
-L LED_RGB D8
+L top-board-rescue:LED_RGB D8
 U 1 1 555223BF
 P 8900 4250
@@
 $EndComp
 $Comp
-L R R38
+L top-board-rescue:R R38
 U 1 1 5551FFDA
 P 8350 1850
@@
 $EndComp
 $Comp
-L R R37
+L top-board-rescue:R R37
 U 1 1 5551FFD4
 P 8350 2050
@@
 $EndComp
 $Comp
-L R R36
+L top-board-rescue:R R36
 U 1 1 5551FFCE
 P 8350 2250
@@
 $EndComp
 $Comp
-L LED_RGB D7
+L top-board-rescue:LED_RGB D7
 U 1 1 5551FFC8
 P 8900 2050
@@
 $EndComp
 $Comp
-L R R35
+L top-board-rescue:R R35
 U 1 1 5551FF9E
 P 8350 2950
@@
 $EndComp
 $Comp
-L R R34
+L top-board-rescue:R R34
 U 1 1 5551FF98
 P 8350 3150
@@
 $EndComp
 $Comp
-L R R33
+L top-board-rescue:R R33
 U 1 1 5551FF92
 P 8350 3350
@@
 $EndComp
 $Comp
-L LED_RGB D6
+L top-board-rescue:LED_RGB D6
 U 1 1 5551FF8C
 P 8900 3150
@@
 $EndComp
 $Comp
-L PCA9685 U5
+L local-components:PCA9685 U5
 U 1 1 5554A9BC
 P 6750 3750
@@
 $EndComp
 $Comp
-L GNDD #PWR083
+L top-board-rescue:GNDD #PWR083
 U 1 1 5554F773
 P 6750 4950
@@
 $EndComp
 $Comp
-L +3.3V #PWR084
+L top-board-rescue:+3.3V #PWR084
 U 1 1 555510C9
 P 6750 2550
@@
 $EndComp
 $Comp
-L GNDD #PWR085
+L top-board-rescue:GNDD #PWR085
 U 1 1 555522F9
 P 6200 4350
@@
 $EndComp
 $Comp
-L GNDD #PWR086
+L top-board-rescue:GNDD #PWR086
 U 1 1 55553181
 P 6150 3600
@@
 $EndComp
 $Comp
-L +3.3V #PWR087
+L top-board-rescue:+3.3V #PWR087
 U 1 1 5555D998
 P 6150 3000
@@
 NoConn ~ 7250 4150
 $Comp
-L GNDD #PWR088
+L top-board-rescue:GNDD #PWR088
 U 1 1 569038AE
 P 9200 3450
@@
 $EndComp
 $Comp
-L GNDD #PWR089
+L top-board-rescue:GNDD #PWR089
 U 1 1 569038D7
 P 9200 4550
@@
 $EndComp
 $Comp
-L GNDD #PWR090
+L top-board-rescue:GNDD #PWR090
 U 1 1 56903ACB
 P 9200 5650
@@
 $EndComp
 $Comp
-L R R47
+L top-board-rescue:R R47
 U 1 1 56905A03
 P 6000 4400
@@
 	6000 3850 6250 3850
 $Comp
-L +3.3V #PWR091
+L top-board-rescue:+3.3V #PWR091
 U 1 1 56906591
 P 5750 4550

Commit message: added logo's and updated gerber files
Parts:
- U5: symbol local-components:PCA9685 -> top-board-rescue:PCA9685-local-components
Changed lines of the file:
@@
 $EndComp
 $Comp
-L local-components:PCA9685 U5
+L top-board-rescue:PCA9685-local-components U5
 U 1 1 5554A9BC
 P 6750 3750
