File: hw-design/top-board/mechanics.sch (KiCad schematic (older format))
At the start: 11 parts

Commit message: Changed SODIM to Marsboard header + added liniar regulator for audio codec
Parts:
- FID1, FID2, FID3, FID4, FID5, FID6: symbol FIDUCIAL -> local-components:FIDUCIAL
- H1, H2, H3, H4, H5: symbol HOLE -> local-components:HOLE
Changed lines of the file:
@@
-EESchema Schematic File Version 2
-LIBS:power
-LIBS:device
-LIBS:conn
-LIBS:regul
-LIBS:74xgxx
-LIBS:local-components
+EESchema Schematic File Version 4
 LIBS:top-board-cache
-EELAYER 25 0
+EELAYER 26 0
 EELAYER END
 $Descr A4 11693 8268
@@
 $EndDescr
 $Comp
-L FIDUCIAL FID1
+L local-components:FIDUCIAL FID1
 U 1 1 55F85886
 P 1300 1150
@@
 $EndComp
 $Comp
-L HOLE H1
+L local-components:HOLE H1
 U 1 1 55F85A35
 P 4900 1150
@@
 $EndComp
 $Comp
-L FIDUCIAL FID2
+L local-components:FIDUCIAL FID2
 U 1 1 55F8753F
 P 1800 1150
@@
 $EndComp
 $Comp
-L FIDUCIAL FID3
+L local-components:FIDUCIAL FID3
 U 1 1 55F87568
 P 2300 1150
@@
 $EndComp
 $Comp
-L FIDUCIAL FID4
+L local-components:FIDUCIAL FID4
 U 1 1 55F87690
 P 2800 1150
@@
 $EndComp
 $Comp
-L FIDUCIAL FID5
+L local-components:FIDUCIAL FID5
 U 1 1 55F87696
 P 3300 1150
@@
 $EndComp
 $Comp
-L FIDUCIAL FID6
+L local-components:FIDUCIAL FID6
 U 1 1 55F8769C
 P 3800 1150
@@
 $EndComp
 $Comp
-L HOLE H2
+L local-components:HOLE H2
 U 1 1 55F87A0A
 P 5200 1150
@@
 $EndComp
 $Comp
-L HOLE H3
+L local-components:HOLE H3
 U 1 1 55F87B0E
 P 5500 1150
@@
 $EndComp
 $Comp
-L HOLE H4
+L local-components:HOLE H4
 U 1 1 55F87B2F
 P 5800 1150
@@
 $EndComp
 $Comp
-L HOLE H5
+L local-components:HOLE H5
 U 1 1 55F87B67
 P 6100 1150

Commit message: added logo's and updated gerber files
Parts:
- FID1, FID2, FID3, FID4, FID5, FID6: symbol local-components:FIDUCIAL -> top-board-rescue:FIDUCIAL-local-components
- H1, H2, H3, H4, H5: symbol local-components:HOLE -> top-board-rescue:HOLE-local-components
Changed lines of the file:
@@
 $EndDescr
 $Comp
-L local-components:FIDUCIAL FID1
+L top-board-rescue:FIDUCIAL-local-components FID1
 U 1 1 55F85886
 P 1300 1150
@@
 $EndComp
 $Comp
-L local-components:HOLE H1
+L top-board-rescue:HOLE-local-components H1
 U 1 1 55F85A35
 P 4900 1150
@@
 $EndComp
 $Comp
-L local-components:FIDUCIAL FID2
+L top-board-rescue:FIDUCIAL-local-components FID2
 U 1 1 55F8753F
 P 1800 1150
@@
 $EndComp
 $Comp
-L local-components:FIDUCIAL FID3
+L top-board-rescue:FIDUCIAL-local-components FID3
 U 1 1 55F87568
 P 2300 1150
@@
 $EndComp
 $Comp
-L local-components:FIDUCIAL FID4
+L top-board-rescue:FIDUCIAL-local-components FID4
 U 1 1 55F87690
 P 2800 1150
@@
 $EndComp
 $Comp
-L local-components:FIDUCIAL FID5
+L top-board-rescue:FIDUCIAL-local-components FID5
 U 1 1 55F87696
 P 3300 1150
@@
 $EndComp
 $Comp
-L local-components:FIDUCIAL FID6
+L top-board-rescue:FIDUCIAL-local-components FID6
 U 1 1 55F8769C
 P 3800 1150
@@
 $EndComp
 $Comp
-L local-components:HOLE H2
+L top-board-rescue:HOLE-local-components H2
 U 1 1 55F87A0A
 P 5200 1150
@@
 $EndComp
 $Comp
-L local-components:HOLE H3
+L top-board-rescue:HOLE-local-components H3
 U 1 1 55F87B0E
 P 5500 1150
@@
 $EndComp
 $Comp
-L local-components:HOLE H4
+L top-board-rescue:HOLE-local-components H4
 U 1 1 55F87B2F
 P 5800 1150
@@
 $EndComp
 $Comp
-L local-components:HOLE H5
+L top-board-rescue:HOLE-local-components H5
 U 1 1 55F87B67
 P 6100 1150
