File: hw-design/bottom-board/Testing Interface.sch (KiCad schematic (older format))
At the start: 16 parts, among them SW2 SW_PUSH, SW3 SW_PUSH

Commit message: added final BOM files
Parts:
- D4, D5, D6: MPN (none) -> LTRBGFSF-ABCB-QKYO-0-0-R18-Z
- R10, R11, R3, R4, R5, R6, R7, R8, R9: MPN (none) -> CRG0603J100R
- R12, R13: MPN (none) -> RMCF0603JT10K0
- SW2, SW3: MPN (none) -> TL3305AF160QG
Changed lines of the file:
@@
 F 2 "LED_SMD:LED_Avago_PLCC6_3x2.8mm" H 2700 1550 50  0001 C CNN
 F 3 "~" H 2700 1550 50  0001 C CNN
+F 4 "LTRBGFSF-ABCB-QKYO-0-0-R18-Z" H 2700 1600 50  0001 C CNN "MPN"
 	1    2700 1600
 	1    0    0    -1
@@
 F 2 "Resistor_SMD:R_0603_1608Metric" V 3130 1600 50  0001 C CNN
 F 3 "" H 3200 1600 50  0001 C CNN
+F 4 "CRG0603J100R" V 3200 1600 50  0001 C CNN "MPN"
 	1    3200 1600
 	0    1    1    0
@@
 F 2 "Resistor_SMD:R_0603_1608Metric" V 3130 1800 50  0001 C CNN
 F 3 "" H 3200 1800 50  0001 C CNN
+F 4 "CRG0603J100R" V 3200 1800 50  0001 C CNN "MPN"
 	1    3200 1800
 	0    1    1    0
@@
 F 2 "LED_SMD:LED_Avago_PLCC6_3x2.8mm" H 2700 2550 50  0001 C CNN
 F 3 "~" H 2700 2550 50  0001 C CNN
+F 4 "LTRBGFSF-ABCB-QKYO-0-0-R18-Z" H 2700 2600 50  0001 C CNN "MPN"
 	1    2700 2600
 	1    0    0    -1
@@
 F 2 "Resistor_SMD:R_0603_1608Metric" V 3130 2400 50  0001 C CNN
 F 3 "" H 3200 2400 50  0001 C CNN
+F 4 "CRG0603J100R" V 3200 2400 50  0001 C CNN "MPN"
 	1    3200 2400
 	0    1    1    0
@@
 F 2 "Resistor_SMD:R_0603_1608Metric" V 3130 2600 50  0001 C CNN
 F 3 "" H 3200 2600 50  0001 C CNN
+F 4 "CRG0603J100R" V 3200 2600 50  0001 C CNN "MPN"
 	1    3200 2600
 	0    1    1    0
@@
 F 2 "Resistor_SMD:R_0603_1608Metric" V 3130 2800 50  0001 C CNN
 F 3 "" H 3200 2800 50  0001 C CNN
+F 4 "CRG0603J100R" V 3200 2800 50  0001 C CNN "MPN"
 	1    3200 2800
 	0    1    1    0
@@
 F 2 "LED_SMD:LED_Avago_PLCC6_3x2.8mm" H 2700 3500 50  0001 C CNN
 F 3 "~" H 2700 3500 50  0001 C CNN
+F 4 "LTRBGFSF-ABCB-QKYO-0-0-R18-Z" H 2700 3550 50  0001 C CNN "MPN"
 	1    2700 3550
 	1    0    0    -1
@@
 F 2 "Resistor_SMD:R_0603_1608Metric" V 3130 3350 50  0001 C CNN
 F 3 "" H 3200 3350 50  0001 C CNN
+F 4 "CRG0603J100R" V 3200 3350 50  0001 C CNN "MPN"
 	1    3200 3350
 	0    1    1    0
@@
 F 2 "Resistor_SMD:R_0603_1608Metric" V 3130 3550 50  0001 C CNN
 F 3 "" H 3200 3550 50  0001 C CNN
+F 4 "CRG0603J100R" V 3200 3550 50  0001 C CNN "MPN"
 	1    3200 3550
 	0    1    1    0
@@
 F 2 "Resistor_SMD:R_0603_1608Metric" V 3130 3750 50  0001 C CNN
 F 3 "" H 3200 3750 50  0001 C CNN
+F 4 "CRG0603J100R" V 3200 3750 50  0001 C CNN "MPN"
 	1    3200 3750
 	0    1    1    0
@@
 F 2 "Resistor_SMD:R_0603_1608Metric" V 3130 1400 50  0001 C CNN
 F 3 "" H 3200 1400 50  0001 C CNN
+F 4 "CRG0603J100R" V 3200 1400 50  0001 C CNN "MPN"
 	1    3200 1400
 	0    1    1    0
@@
 F 2 "Resistor_SMD:R_0603_1608Metric" V 7030 1450 50  0001 C CNN
 F 3 "" H 7100 1450 50  0001 C CNN
+F 4 "RMCF0603JT10K0" V 7100 1450 50  0001 C CNN "MPN"
 	1    7100 1450
 	-1   0    0    1
@@
 F 2 "Button_Switch_SMD:SW_SPST_TL3305A" H 6300 1863 50  0000 C CNN
 F 3 "" H 6300 1700 50  0000 C CNN
+F 4 "TL3305AF160QG" H 6300 1700 50  0001 C CNN "MPN"
 	1    6300 1700
 	1    0    0    -1
@@
 F 2 "Resistor_SMD:R_0603_1608Metric" V 7030 2550 50  0001 C CNN
 F 3 "" H 7100 2550 50  0001 C CNN
+F 4 "RMCF0603JT10K0" V 7100 2550 50  0001 C CNN "MPN"
 	1    7100 2550
 	-1   0    0    1
@@
 F 2 "Button_Switch_SMD:SW_SPST_TL3305A" H 6300 2963 50  0000 C CNN
 F 3 "" H 6300 2800 50  0000 C CNN
+F 4 "TL3305AF160QG" H 6300 2800 50  0001 C CNN "MPN"
 	1    6300 2800
 	1    0    0    -1
