File: hw-design/bottom-board/USB device.sch (KiCad schematic (older format))
At the start: 8 parts, among them P1 USB_B-RESCUE-bottom-board

Commit message: added final BOM files
Parts:
- C10, C8: MPN (none) -> C1608X7R1E104K080AA
- C9: MPN (none) -> GRM219R61E106KA12D
- D3: MPN (none) -> PRTR5V0U2X,215
- L1: MPN (none) -> 742792651
- P1: MPN (none) -> 61729-1011BLF
- R1: MPN (none) -> CRGCQ0603F5K6
- R2: MPN (none) -> RMCF0603JT10K0
Changed lines of the file:
@@
 F 0 "P1" H 4628 2775 50  0000 C CNN
 F 1 "USB_B-RESCUE-bottom-board" H 4628 2684 50  0000 C CNN
-F 2 "Connector_USB:USB_B_OST_USB-B1HSxx_Horizontal" H 4500 2800 50  0000 C CNN
+F 2 "Connector_USB:USB_B_OST_USB-B1HSxx_Horizontal" H 4500 2800 50  0001 C CNN
 F 3 "" V 4550 2350 50  0000 C CNN
+F 4 "61729-1011BLF" H 4600 2450 50  0001 C CNN "MPN"
 	1    4600 2450
 	1    0    0    -1
@@
 F 2 "Resistor_SMD:R_0603_1608Metric" V 3830 3000 50  0001 C CNN
 F 3 "" H 3900 3000 50  0001 C CNN
+F 4 "CRGCQ0603F5K6" H 3900 3000 50  0001 C CNN "MPN"
 	1    3900 3000
 	1    0    0    -1
@@
 F 2 "Resistor_SMD:R_0603_1608Metric" V 3830 3500 50  0001 C CNN
 F 3 "" H 3900 3500 50  0001 C CNN
+F 4 "RMCF0603JT10K0" H 3900 3500 50  0001 C CNN "MPN"
 	1    3900 3500
 	1    0    0    -1
@@
 F 2 "Capacitor_SMD:C_0805_2012Metric" H 3200 3500 50  0001 C CNN
 F 3 "" H 3200 3500 50  0001 C CNN
+F 4 "C1608X7R1E104K080AA" H 3200 3500 50  0001 C CNN "MPN"
 	1    3200 3500
 	1    0    0    -1
@@
 F 2 "Capacitor_SMD:C_0805_2012Metric" H 4350 3250 50  0001 C CNN
 F 3 "" H 4350 3250 50  0001 C CNN
+F 4 "GRM219R61E106KA12D" H 4350 3250 50  0001 C CNN "MPN"
 	1    4350 3250
 	1    0    0    -1
@@
 F 2 "Package_TO_SOT_SMD:SOT-143_Handsoldering" H 5600 3650 50  0001 C CNN
 F 3 "" H 5600 3650 50  0001 C CNN
+F 4 "PRTR5V0U2X,215" H 5550 3700 50  0001 C CNN "MPN"
 	1    5550 3700
 	1    0    0    -1
@@
 F 2 "Capacitor_SMD:C_0805_2012Metric" H 4950 3700 50  0001 C CNN
 F 3 "" H 4950 3700 50  0001 C CNN
+F 4 "C1608X7R1E104K080AA" H 4950 3700 50  0001 C CNN "MPN"
 	1    4950 3700
 	1    0    0    -1
@@
 F 2 "Capacitor_SMD:C_0805_2012Metric" H 5200 2650 50  0001 C CNN
 F 3 "" H 5200 2650 50  0001 C CNN
+F 4 "742792651" H 5200 2650 50  0001 C CNN "MPN"
 	1    5200 2650
 	1    0    0    -1
