File: hw-design/bottom-board/connectors.sch (KiCad schematic (older format))
At the start: 7 parts, among them P5 BARREL_JACK, P6 HMI_POWER, P8 HMI_DATA, P9 SERIAL_DEBUG

Commit message: added final BOM files
Parts:
- C55: footprint Capacitors_SMD:C_0603 -> Capacitor_SMD:C_0603_1608Metric
- R72, R73: footprint Resistors_SMD:R_0603 -> Resistor_SMD:R_0603_1608Metric
Changed lines of the file:
@@
 Sheet 4 7
 Title "MOD Duo -HMI testing board"
-Date ""
+Date "2019-08-16"
 Rev "1.0"
 Comp "MOD Devices GmbH"
@@
 F 2 "Pin_Headers:Pin_Header_Straight_1x03" H 9750 2650 60  0001 C CNN
 F 3 "" H 9750 2650 60  0000 C CNN
+F 4 "~" H 9750 2650 50  0001 C CNN "MPN "
 	1    9750 2650
 	1    0    0    -1
@@
 F 0 "C55" H 2700 1550 50  0000 L CNN
 F 1 "100nF" H 2650 1450 50  0000 L CNN
-F 2 "Capacitors_SMD:C_0603" H 2600 1550 60  0001 C CNN
+F 2 "Capacitor_SMD:C_0603_1608Metric" H 2600 1550 60  0001 C CNN
 F 3 "" H 2600 1550 60  0000 C CNN
 F 4 "C1608X7R1E104K080AA" H 0   0   50  0001 C CNN "MPN"
@@
 F 0 "R72" V 8500 1300 50  0000 L CNN
 F 1 "100R" V 8500 1600 50  0000 L CNN
-F 2 "Resistors_SMD:R_0603" H 8550 1500 60  0001 C CNN
+F 2 "Resistor_SMD:R_0603_1608Metric" H 8550 1500 60  0001 C CNN
 F 3 "" H 8550 1500 60  0000 C CNN
 F 4 "RMCF0603JT100R" H -200 -3850 50  0001 C CNN "MPN"
@@
 F 0 "R73" V 8500 1400 50  0000 L CNN
 F 1 "100R" V 8500 1700 50  0000 L CNN
-F 2 "Resistors_SMD:R_0603" H 8550 1600 60  0001 C CNN
+F 2 "Resistor_SMD:R_0603_1608Metric" H 8550 1600 60  0001 C CNN
 F 3 "" H 8550 1600 60  0000 C CNN
 F 4 "RMCF0603JT100R" H -200 -3750 50  0001 C CNN "MPN"
