File: hw-design/bottom-board/connectors.sch (KiCad schematic (older format))
At the start: 25 parts, among them J1 JACK_TRS_6PINS, J2 JACK_TRS_6PINS, J3 JACK_TRS_6PINS, J4 JACK_TRS_6PINS, J5 JACK_TRS_6PINS, J6 RJ45_LEDS, P5 BARREL_JACK, P6 HMI_POWER, P7 SD_CARD, P8 HMI_DATA, P9 SERIAL_DEBUG

Commit message: Changed SODIM to Marsboard header + added liniar regulator for audio codec
Parts:
- removed P7: SD_CARD, Pin_Headers:Pin_Header_Straight_1x10, symbol bottom-board-rescue:CONN_01X10
- removed R64, R65, R66, R67, R68, R69, R70: 10k, Resistors_SMD:R_0603, symbol bottom-board-rescue:R_Small
Connections:
- net labels removed: +3.3V, SD0_CLK, SD0_CMD, SD0_D0, SD0_D1, SD0_D2, SD0_D3, SD0_DETECT
- wire segments 107 -> 94
- no-connect marks 14 -> 13
Other:
- note removed: "SD CARD"

Commit message: updated footprints and MPN's
Parts:
- C55, C57: footprint Capacitors_SMD:C_0603 -> Capacitor_SMD:C_0603_1608Metric
- C56: footprint Capacitors_SMD:c_elec_5x5.3 -> Capacitor_SMD:CP_Elec_5x5.3
- J1, J2, J3, J4, J5: footprint Connect:NMJ6HCD2 -> Connector_Audio:Jack_3.5mm_Neutrik_NMJ6HCD2_Horizontal; symbol bottom-board-rescue:JACK_TRS_6PINS -> Connector:AudioJack3_Switch
- J6: footprint Connect:RJHSE538X -> Connector_RJ:RJ45_Amphenol_RJHSE538X
- P5: footprint Connect:BARREL_JACK -> Connector_BarrelJack:BarrelJack_Horizontal
- P9: footprint Pin_Headers:Pin_Header_Straight_1x03 -> Connector_PinHeader_2.54mm:PinHeader_1x03_P2.54mm_Vertical
- R72, R73, R76, R77: footprint Resistors_SMD:R_0603 -> Resistor_SMD:R_0603_1608Metric
Connections:
- net GNDA: now also J1.R, J1.S, J1.TN, J2.R, J2.S, J2.TN, J3.S, J4.S, J5.S; no longer J1.1 (S), J1.3 (R), J1.5 (TN), J2.1 (S), J2.3 (R), J2.5 (TN), J3.1 (S), J4.1 (S), J5.1 (S)
- net HP_LEFT: now also J5.T; no longer J5.2 (T)
- net HP_RIGHT: now also J5.R; no longer J5.3 (R)
- net LEFT_AUDIO_INPUT: now also J1.T; no longer J1.2 (T)
- net LEFT_AUDIO_OUTPUT_RING: now also J3.R; no longer J3.3 (R)
- net LEFT_AUDIO_OUTPUT_TIP: now also J3.T; no longer J3.2 (T)
- net RIGHT_AUDIO_INPUT: now also J2.T; no longer J2.2 (T)
- net RIGHT_AUDIO_OUTPUT_RING: now also J4.R; no longer J4.3 (R)
- net RIGHT_AUDIO_OUTPUT_TIP: now also J4.T; no longer J4.2 (T)
