File: hw-design/bottom-board/power.sch (KiCad schematic (older format))
At the start: 18 parts, among them U1 MURATA 5V, U2 LD1117S50TR_SOT223

Commit message: updated footprints and MPN's
Parts:
- C1, C10, C4, C5, C9: footprint Capacitors_SMD:C_0603 -> Capacitor_SMD:C_0603_1608Metric
- C11, C8: MPN UWX1E100MCL1GB -> GRM219R61E106KA12D
- C3, C7: footprint Capacitors_SMD:C_0805 -> Capacitor_SMD:C_0805_2012Metric
Changed lines of the file:
@@
 EESchema Schematic File Version 4
 LIBS:bottom-board-cache
-EELAYER 26 0
+EELAYER 29 0
 EELAYER END
 $Descr A4 11693 8268
@@
 F 0 "C1" H 4000 3150 50  0000 L CNN
 F 1 "100nF" H 3700 2950 50  0000 L CNN
-F 2 "Capacitors_SMD:C_0603" H 3988 2900 30  0001 C CNN
+F 2 "Capacitor_SMD:C_0603_1608Metric" H 3988 2900 30  0001 C CNN
 F 3 "" H 3950 3050 60  0000 C CNN
 F 4 "C1608X7R1E104K080AA" H 800 250 50  0001 C CNN "MPN"
@@
 F 0 "C9" H 6900 3150 50  0000 L CNN
 F 1 "100nF" H 6600 2950 50  0000 L CNN
-F 2 "Capacitors_SMD:C_0603" H 6888 2900 30  0001 C CNN
+F 2 "Capacitor_SMD:C_0603_1608Metric" H 6888 2900 30  0001 C CNN
 F 3 "" H 6850 3050 60  0000 C CNN
 F 4 "C1608X7R1E104K080AA" H 1300 250 50  0001 C CNN "MPN"
@@
 F 0 "C10" H 8050 3150 50  0000 L CNN
 F 1 "100nF" H 7750 2950 50  0000 L CNN
-F 2 "Capacitors_SMD:C_0603" H 8038 2900 30  0001 C CNN
+F 2 "Capacitor_SMD:C_0603_1608Metric" H 8038 2900 30  0001 C CNN
 F 3 "" H 8000 3050 60  0000 C CNN
 F 4 "C1608X7R1E104K080AA" H 1200 250 50  0001 C CNN "MPN"
@@
 F 0 "C4" H 5350 3150 50  0000 L CNN
 F 1 "100nF" H 5050 2950 50  0000 L CNN
-F 2 "Capacitors_SMD:C_0603" H 5338 2900 30  0001 C CNN
+F 2 "Capacitor_SMD:C_0603_1608Metric" H 5338 2900 30  0001 C CNN
 F 3 "" H 5300 3050 60  0000 C CNN
 F 4 "C1608X7R1E104K080AA" H 800 250 50  0001 C CNN "MPN"
@@
 F 0 "C5" H 5550 4950 50  0000 L CNN
 F 1 "100nF" H 5250 4750 50  0000 L CNN
-F 2 "Capacitors_SMD:C_0603" H 5538 4700 30  0001 C CNN
+F 2 "Capacitor_SMD:C_0603_1608Metric" H 5538 4700 30  0001 C CNN
 F 3 "" H 5500 4850 60  0000 C CNN
 F 4 "C1608X7R1E104K080AA" H -1600 250 50  0001 C CNN "MPN"
@@
 F 0 "C7" H 5900 4950 50  0000 L CNN
 F 1 "10uF" H 5650 4750 50  0000 L CNN
-F 2 "Capacitors_SMD:C_0805" H 5850 4850 60  0001 C CNN
+F 2 "Capacitor_SMD:C_0805_2012Metric" H 5850 4850 60  0001 C CNN
 F 3 "" H 5850 4850 60  0000 C CNN
 F 4 "GRM219R61E106KA12D" H 550 -500 50  0001 C CNN "MPN"
@@
 F 2 "Capacitor_SMD:C_0805_2012Metric" H 6500 3050 60  0001 C CNN
 F 3 "" H 6500 3050 60  0000 C CNN
-F 4 "UWX1E100MCL1GB" H 1400 1550 50  0001 C CNN "MPN"
+F 4 "GRM219R61E106KA12D" H 1400 1550 50  0001 C CNN "MPN"
 	1    6500 3050
 	1    0    0    -1
@@
 F 0 "C3" H 4350 4950 50  0000 L CNN
 F 1 "10uF" H 4100 4750 50  0000 L CNN
-F 2 "Capacitors_SMD:C_0805" H 4300 4850 60  0001 C CNN
+F 2 "Capacitor_SMD:C_0805_2012Metric" H 4300 4850 60  0001 C CNN
 F 3 "" H 4300 4850 60  0000 C CNN
 F 4 "GRM219R61E106KA12D" H -1000 -500 50  0001 C CNN "MPN"
@@
 F 2 "Capacitor_SMD:C_0805_2012Metric" H 8350 3050 60  0001 C CNN
 F 3 "" H 8350 3050 60  0000 C CNN
-F 4 "UWX1E100MCL1GB" H 3250 1550 50  0001 C CNN "MPN"
+F 4 "GRM219R61E106KA12D" H 3250 1550 50  0001 C CNN "MPN"
 	1    8350 3050
 	1    0    0    -1
