File: hw-design/bottom-board/audio-headphones.sch (KiCad schematic (older format))
At the start: 12 parts, among them U9 LM4811

Commit message: Changed SODIM to Marsboard header + added liniar regulator for audio codec
Parts:
- removed CA21, CA22: 1uF, Capacitors_SMD:C_0805, symbol bottom-board-rescue:C_Small
- added C32, C36, C61: 10uF, Capacitor_SMD:C_Elec_5x5.4, symbol bottom-board-rescue:CP_Small
- added C33: 100nF, Capacitor_SMD:C_0402_1005Metric, symbol bottom-board-rescue:C_Small
- CA24, CA25: footprint Capacitors_SMD:c_elec_5x5.3 -> Capacitor_SMD:CP_Elec_6.3x7.7
Connections:
- wire segments 36 -> 49
Changed lines of the file:
@@
-$EndComp
-$Comp
-L bottom-board-rescue:C_Small CA22
-U 1 1 550D4F2F
-P 4450 2750
-F 0 "CA22" V 4500 2800 50  0000 L CNN
-F 1 "1uF" V 4400 2800 50  0000 L CNN
-F 2 "Capacitors_SMD:C_0805" H 4450 2750 60  0001 C CNN
-F 3 "" H 4450 2750 60  0000 C CNN
-F 4 "C2012X7R1E105K125AB" H 0   1050 50  0001 C CNN "MPN"
-	1    4450 2750
-	0    1    1    0
 $EndComp
 $Comp
@@
 F 0 "CA25" V 6700 3650 50  0000 L CNN
 F 1 "100uF" V 6850 3500 50  0000 L CNN
-F 2 "Capacitors_SMD:c_elec_5x5.3" H 6750 3550 60  0001 C CNN
+F 2 "Capacitor_SMD:CP_Elec_6.3x7.7" H 6750 3550 60  0001 C CNN
 F 3 "" H 6750 3550 60  0000 C CNN
 F 4 "EEE-FT1C101AR" H 0   1050 50  0001 C CNN "MPN"
@@
 F 0 "CA24" V 6700 2850 50  0000 L CNN
 F 1 "100uF" V 6850 2650 50  0000 L CNN
-F 2 "Capacitors_SMD:c_elec_5x5.3" H 6750 2750 60  0001 C CNN
+F 2 "Capacitor_SMD:CP_Elec_6.3x7.7" H 6750 2750 60  0001 C CNN
 F 3 "" H 6750 2750 60  0000 C CNN
 F 4 "EEE-FT1C101AR" H 0   1050 50  0001 C CNN "MPN"
@@
 $EndComp
 $Comp
-L power:GNDA #PWR0119
+L bottom-board-rescue:GNDA-power #PWR0119
 U 1 1 550C34F1
 P 7000 4000
+AR Path="/550C34F1" Ref="#PWR0119"  Part="1"
+AR Path="/54F72F64/550C34F1" Ref="#PWR0119"  Part="1"
 F 0 "#PWR0119" H 7000 3750 50  0001 C CNN
 F 1 "GNDA" H 7000 3850 50  0000 C CNN
@@
 $EndComp
 $Comp
-L power:GNDA #PWR0120
+L bottom-board-rescue:GNDA-power #PWR0120
 U 1 1 550C353B
 P 7000 3200
+AR Path="/550C353B" Ref="#PWR0120"  Part="1"
+AR Path="/54F72F64/550C353B" Ref="#PWR0120"  Part="1"
 F 0 "#PWR0120" H 7000 2950 50  0001 C CNN
 F 1 "GNDA" H 7000 3050 50  0000 C CNN
@@
 	1    7000 3200
 	-1   0    0    -1
-$EndComp
-$Comp
-L bottom-board-rescue:C_Small CA21
-U 1 1 551BDF86
-P 4050 2850
-F 0 "CA21" V 4100 2900 50  0000 L CNN
-F 1 "1uF" V 4000 2900 50  0000 L CNN
-F 2 "Capacitors_SMD:C_0805" H 4050 2850 60  0001 C CNN
-F 3 "" H 4050 2850 60  0000 C CNN
-F 4 "C2012X7R1E105K125AB" H 0   1050 50  0001 C CNN "MPN"
-	1    4050 2850
-	0    1    1    0
 $EndComp
 Text GLabel 4150 3050 0    50   Input ~ 0
@@
 Text GLabel 7250 2750 2    50   Output ~ 0
 HP_LEFT
-Text GLabel 3650 2850 0    50   Input ~ 0
-CODEC_AUX_B
-Text GLabel 3650 2750 0    50   Input ~ 0
-CODEC_AUX_A
 Wire Wire Line
 	4600 3350 4600 3450
@@
 Wire Wire Line
 	4550 2750 4750 2750
-Wire Wire Line
-	4750 2850 4150 2850
-Wire Wire Line
-	3650 2850 3950 2850
-Wire Wire Line
-	3650 2750 4350 2750
 Connection ~ 7000 3550
 Connection ~ 7000 2750
@@
 Connection ~ 5350 2300
 $Comp
-L power:GNDA #PWR0121
+L bottom-board-rescue:GNDA-power #PWR0121
 U 1 1 5570B05D
 P 5350 4100
+AR Path="/5570B05D" Ref="#PWR0121"  Part="1"
+AR Path="/54F72F64/5570B05D" Ref="#PWR0121"  Part="1"
 F 0 "#PWR0121" H 5350 3850 50  0001 C CNN
 F 1 "GNDA" H 5350 3950 50  0000 C CNN
@@
 $EndComp
 $Comp
-L power:GNDA #PWR0122
+L bottom-board-rescue:GNDA-power #PWR0122
 U 1 1 5570B0BB
 P 4600 3450
+AR Path="/5570B0BB" Ref="#PWR0122"  Part="1"
+AR Path="/54F72F64/5570B0BB" Ref="#PWR0122"  Part="1"
 F 0 "#PWR0122" H 4600 3200 50  0001 C CNN
 F 1 "GNDA" H 4600 3300 50  0000 C CNN
@@
 $EndComp
 $Comp
-L power:+5VA #PWR0123
+L bottom-board-rescue:+5VA-power #PWR0123
 U 1 1 5570BCEC
 P 5350 1950
@@
 $EndComp
 $Comp
-L power:GNDA #PWR0124
+L bottom-board-rescue:GNDA-power #PWR0124
 U 1 1 5570D8B7
 P 5850 2350
+AR Path="/5570D8B7" Ref="#PWR0124"  Part="1"
+AR Path="/54F72F64/5570D8B7" Ref="#PWR0124"  Part="1"
 F 0 "#PWR0124" H 5850 2100 50  0001 C CNN
 F 1 "GNDA" H 5850 2200 50  0000 C CNN
@@
 Wire Wire Line
 	5850 2300 5850 2350
+Text GLabel 3250 2700 0    50   Input ~ 0
+CODEC_AUX_A
+Text GLabel 3300 2850 0    50   Input ~ 0
+CODEC_AUX_B
+$Comp
+L bottom-board-rescue:CP_Small C61
+U 1 1 5C9975FC
+P 3750 2700
+F 0 "C61" V 3700 2650 50  0000 R CNN
+F 1 "10uF" V 3850 2750 50  0000 R CNN
+F 2 "Capacitor_SMD:C_Elec_5x5.4" H 3750 2700 60  0001 C CNN
+F 3 "" H 3750 2700 60  0000 C CNN
+F 4 "UWX1E100MCL1GB" H -3000 200 50  0001 C CNN "MPN"
+	1    3750 2700
+	0    -1   -1   0
+$EndComp
+$Comp
+L bottom-board-rescue:CP_Small C32
+U 1 1 5C997652
+P 3750 2850
+F 0 "C32" V 3700 2800 50  0000 R CNN
+F 1 "10uF" V 3850 2900 50  0000 R CNN
+F 2 "Capacitor_SMD:C_Elec_5x5.4" H 3750 2850 60  0001 C CNN
+F 3 "" H 3750 2850 60  0000 C CNN
+F 4 "UWX1E100MCL1GB" H -3000 350 50  0001 C CNN "MPN"
+	1    3750 2850
+	0    -1   -1   0
+$EndComp
+Wire Wire Line
+	3850 2700 4550 2700
+Wire Wire Line
+	4550 2700 4550 2750
+Wire Wire Line
+	3850 2850 4750 2850
+$Comp
+L bottom-board-rescue:C_Small C?
+U 1 1 5C99E218
+P 4950 1250
+AR Path="/54F72B97/5C99E218" Ref="C?"  Part="1"
+AR Path="/54F72F64/5C99E218" Ref="C33"  Part="1"
+F 0 "C33" V 4900 1050 50  0000 L CNN
+F 1 "100nF" V 4900 1300 50  0000 L CNN
+F 2 "Capacitor_SMD:C_0402_1005Metric" H 4950 1250 60  0001 C CNN
+F 3 "" H 4950 1250 60  0000 C CNN
+F 4 "C1005X7R1E104K050BB" H -350 -4100 50  0001 C CNN "MPN"
+	1    4950 1250
+	1    0    0    -1
+$EndComp
+Wire Wire Line
+	5100 1150 5100 1000
+Wire Wire Line
+	5100 1000 4950 1000
+Wire Wire Line
+	4950 1350 4950 1450
+Wire Wire Line
+	5100 1350 5100 1450
+$Comp
+L bottom-board-rescue:CP_Small C?
+U 1 1 5C99E225
+P 5100 1250
+AR Path="/54F72B97/5C99E225" Ref="C?"  Part="1"
+AR Path="/54F72F64/5C99E225" Ref="C36"  Part="1"
+F 0 "C36" V 5150 1050 50  0000 L CNN
+F 1 "10uF" V 5150 1300 50  0000 L CNN
+F 2 "Capacitor_SMD:C_Elec_5x5.4" H 5100 1250 60  0001 C CNN
+F 3 "" H 5100 1250 60  0000 C CNN
+F 4 "UWX1E100MCL1GB" H 0   -250 50  0001 C CNN "MPN"
+	1    5100 1250
+	1    0    0    -1
+$EndComp
+Wire Wire Line
+	4950 1000 4950 1150
+Wire Wire Line
+	4950 1450 5050 1450
+$Comp
+L bottom-board-rescue:GNDA-power #PWR?
+U 1 1 5C99E22E
+P 5000 1500
+AR Path="/54F72B97/5C99E22E" Ref="#PWR?"  Part="1"
+AR Path="/54F72F64/5C99E22E" Ref="#PWR0142"  Part="1"
+AR Path="/5C99E22E" Ref="#PWR0142"  Part="1"
+F 0 "#PWR0142" H 5000 1250 50  0001 C CNN
+F 1 "GNDA" H 5000 1350 50  0000 C CNN
+F 2 "" H 5000 1500 60  0000 C CNN
+F 3 "" H 5000 1500 60  0000 C CNN
+	1    5000 1500
+	1    0    0    -1
+$EndComp
+Wire Wire Line
+	5000 1500 5000 1400
+Wire Wire Line
+	5000 1400 5050 1400
+Wire Wire Line
+	5050 1400 5050 1450
+Connection ~ 5050 1450
+Wire Wire Line
+	5050 1450 5100 1450
+$Comp
+L bottom-board-rescue:+5VA-power #PWR0143
+U 1 1 5C99F854
+P 4950 900
+F 0 "#PWR0143" H 4950 750 50  0001 C CNN
+F 1 "+5VA" H 4950 1040 50  0000 C CNN
+F 2 "" H 4950 900 60  0000 C CNN
+F 3 "" H 4950 900 60  0000 C CNN
+	1    4950 900
+	1    0    0    -1
+$EndComp
+Wire Wire Line
+	4950 900  4950 1000
+Connection ~ 4950 1000
+Wire Wire Line
+	3250 2700 3650 2700
+Wire Wire Line
+	3300 2850 3650 2850
 $EndSCHEMATC

Commit message: updated footprints and MPN's
Parts:
- C32, C36, C61: footprint Capacitor_SMD:C_Elec_5x5.4 -> Capacitor_SMD:CP_Elec_5x5.3
- C33: footprint Capacitor_SMD:C_0402_1005Metric -> Capacitor_SMD:C_0603_1608Metric; MPN C1005X7R1E104K050BB -> C1608X7R1E104K080AA
- C46, CA23: footprint Capacitors_SMD:c_elec_5x5.3 -> Capacitor_SMD:CP_Elec_5x5.3
- C47: footprint Capacitors_SMD:C_0603 -> Capacitor_SMD:C_0603_1608Metric
- CA24, CA25: MPN EEE-FT1C101AR -> UWT1E101MCL1GS
- R40, R41, RA39, RA40: footprint Resistors_SMD:R_0603 -> Resistor_SMD:R_0603_1608Metric
Changed lines of the file:
@@
 EESchema Schematic File Version 4
 LIBS:bottom-board-cache
-EELAYER 26 0
+EELAYER 29 0
 EELAYER END
 $Descr A4 11693 8268
@@
 F 0 "CA23" H 5650 3850 50  0000 L CNN
 F 1 "10uF" H 5650 3750 50  0000 L CNN
-F 2 "Capacitors_SMD:c_elec_5x5.3" H 5550 3850 60  0001 C CNN
+F 2 "Capacitor_SMD:CP_Elec_5x5.3" H 5550 3850 60  0001 C CNN
 F 3 "" H 5550 3850 60  0000 C CNN
 F 4 "UWX1E100MCL1GB" H 0   1050 50  0001 C CNN "MPN"
@@
 F 0 "C47" V 5650 2250 50  0000 R CNN
 F 1 "100nF" V 5500 2350 50  0000 R CNN
-F 2 "Capacitors_SMD:C_0603" H 5600 2300 60  0001 C CNN
+F 2 "Capacitor_SMD:C_0603_1608Metric" H 5600 2300 60  0001 C CNN
 F 3 "" H 5600 2300 60  0000 C CNN
 F 4 "C1608X7R1E104K080AA" H 50  1050 50  0001 C CNN "MPN"
@@
 F 2 "Capacitor_SMD:CP_Elec_6.3x7.7" H 6750 3550 60  0001 C CNN
 F 3 "" H 6750 3550 60  0000 C CNN
-F 4 "EEE-FT1C101AR" H 0   1050 50  0001 C CNN "MPN"
+F 4 "UWT1E101MCL1GS" H 0   1050 50  0001 C CNN "MPN"
 	1    6750 3550
 	0    -1   -1   0
@@
 F 0 "RA40" H 7050 3850 50  0000 L CNN
 F 1 "75k" H 7050 3750 50  0000 L CNN
-F 2 "Resistors_SMD:R_0603" H 7000 3800 60  0001 C CNN
+F 2 "Resistor_SMD:R_0603_1608Metric" H 7000 3800 60  0001 C CNN
 F 3 "" H 7000 3800 60  0000 C CNN
 F 4 "ERA-3AEB753V" H 0   1050 50  0001 C CNN "MPN"
@@
 F 2 "Capacitor_SMD:CP_Elec_6.3x7.7" H 6750 2750 60  0001 C CNN
 F 3 "" H 6750 2750 60  0000 C CNN
-F 4 "EEE-FT1C101AR" H 0   1050 50  0001 C CNN "MPN"
+F 4 "UWT1E101MCL1GS" H 0   1050 50  0001 C CNN "MPN"
 	1    6750 2750
 	0    -1   -1   0
@@
 F 0 "RA39" H 7050 3050 50  0000 L CNN
 F 1 "75k" H 7050 2950 50  0000 L CNN
-F 2 "Resistors_SMD:R_0603" H 7000 3000 60  0001 C CNN
+F 2 "Resistor_SMD:R_0603_1608Metric" H 7000 3000 60  0001 C CNN
 F 3 "" H 7000 3000 60  0000 C CNN
 F 4 "ERA-3AEB753V" H 0   1050 50  0001 C CNN "MPN"
@@
 F 0 "C46" V 5550 2000 50  0000 R CNN
 F 1 "10uF" V 5700 2100 50  0000 R CNN
-F 2 "Capacitors_SMD:c_elec_5x5.3" H 5600 2050 60  0001 C CNN
+F 2 "Capacitor_SMD:CP_Elec_5x5.3" H 5600 2050 60  0001 C CNN
 F 3 "" H 5600 2050 60  0000 C CNN
 F 4 "UWX1E100MCL1GB" H -1150 -450 50  0001 C CNN "MPN"
@@
 F 0 "R40" V 4400 2850 50  0000 L CNN
 F 1 "22R" V 4400 3150 50  0000 L CNN
-F 2 "Resistors_SMD:R_0603" H 4450 3050 60  0001 C CNN
+F 2 "Resistor_SMD:R_0603_1608Metric" H 4450 3050 60  0001 C CNN
 F 3 "" H 4450 3050 60  0000 C CNN
 F 4 "RMCF0603JT22R0" H 150 700 50  0001 C CNN "MPN"
@@
 F 0 "R41" V 4400 2950 50  0000 L CNN
 F 1 "22R" V 4400 3250 50  0000 L CNN
-F 2 "Resistors_SMD:R_0603" H 4450 3150 60  0001 C CNN
+F 2 "Resistor_SMD:R_0603_1608Metric" H 4450 3150 60  0001 C CNN
 F 3 "" H 4450 3150 60  0000 C CNN
 F 4 "RMCF0603JT22R0" H 150 800 50  0001 C CNN "MPN"
@@
 F 0 "C61" V 3700 2650 50  0000 R CNN
 F 1 "10uF" V 3850 2750 50  0000 R CNN
-F 2 "Capacitor_SMD:C_Elec_5x5.4" H 3750 2700 60  0001 C CNN
+F 2 "Capacitor_SMD:CP_Elec_5x5.3" H 3750 2700 60  0001 C CNN
 F 3 "" H 3750 2700 60  0000 C CNN
 F 4 "UWX1E100MCL1GB" H -3000 200 50  0001 C CNN "MPN"
@@
 F 0 "C32" V 3700 2800 50  0000 R CNN
 F 1 "10uF" V 3850 2900 50  0000 R CNN
-F 2 "Capacitor_SMD:C_Elec_5x5.4" H 3750 2850 60  0001 C CNN
+F 2 "Capacitor_SMD:CP_Elec_5x5.3" H 3750 2850 60  0001 C CNN
 F 3 "" H 3750 2850 60  0000 C CNN
 F 4 "UWX1E100MCL1GB" H -3000 350 50  0001 C CNN "MPN"
@@
 F 0 "C33" V 4900 1050 50  0000 L CNN
 F 1 "100nF" V 4900 1300 50  0000 L CNN
-F 2 "Capacitor_SMD:C_0402_1005Metric" H 4950 1250 60  0001 C CNN
+F 2 "Capacitor_SMD:C_0603_1608Metric" H 4950 1250 60  0001 C CNN
 F 3 "" H 4950 1250 60  0000 C CNN
-F 4 "C1005X7R1E104K050BB" H -350 -4100 50  0001 C CNN "MPN"
+F 4 "C1608X7R1E104K080AA" H -350 -4100 50  0001 C CNN "MPN"
 	1    4950 1250
 	1    0    0    -1
@@
 F 0 "C36" V 5150 1050 50  0000 L CNN
 F 1 "10uF" V 5150 1300 50  0000 L CNN
-F 2 "Capacitor_SMD:C_Elec_5x5.4" H 5100 1250 60  0001 C CNN
+F 2 "Capacitor_SMD:CP_Elec_5x5.3" H 5100 1250 60  0001 C CNN
 F 3 "" H 5100 1250 60  0000 C CNN
 F 4 "UWX1E100MCL1GB" H 0   -250 50  0001 C CNN "MPN"
