File: hw-design/bottom-board/control-chain.sch (KiCad schematic (older format))
At the start: 15 parts, among them Q14 BSS84, Q15 BSS84, U12 ISL83491

Commit message: Changed SODIM to Marsboard header + added liniar regulator for audio codec
Connections:
- wire segments 44 -> 55
Changed lines of the file:
@@
 $EndComp
 $Comp
-L power:GNDD #PWR0144
+L bottom-board-rescue:GNDD-power #PWR0144
 U 1 1 550C7BE5
 P 5850 2800
@@
 $EndComp
 $Comp
-L power:GNDD #PWR0145
+L bottom-board-rescue:GNDD-power #PWR0145
 U 1 1 550C7C57
 P 5500 4450
@@
 $EndComp
 $Comp
-L power:+3.3V #PWR0146
+L bottom-board-rescue:+3.3V-power #PWR0146
 U 1 1 551A1FF5
 P 5300 2650
@@
 	4750 3300 4900 3300
 Wire Wire Line
-	4700 3800 4900 3800
+	4700 3800 4800 3800
 Wire Wire Line
 	5850 2800 5850 2750
@@
 	5850 2750 5750 2750
 Wire Wire Line
-	4350 3300 4550 3300
+	4350 3300 4450 3300
 Wire Wire Line
 	4350 3800 4500 3800
 Wire Wire Line
-	5300 2650 5300 2900
+	5300 2650 5300 2750
 Wire Wire Line
 	5200 2900 5200 2750
 Wire Wire Line
-	5500 4300 5500 4450
+	5500 4300 5500 4400
 Wire Wire Line
 	5600 4300 5600 4400
@@
 	5900 3400 6000 3400
 Wire Wire Line
-	6450 3150 6950 3150
+	6450 3150 6650 3150
 Wire Wire Line
 	6450 3150 6450 3200
@@
 	6450 3200 6200 3200
 Wire Wire Line
-	6450 3450 6950 3450
+	6450 3450 6650 3450
 Wire Wire Line
 	6450 3450 6450 3400
@@
 	6450 3900 6600 3900
 Wire Wire Line
-	4350 3500 4900 3500
-Wire Wire Line
-	4350 4000 4900 4000
+	4350 3500 4800 3500
+Wire Wire Line
+	4350 4000 4800 4000
 Connection ~ 5300 2750
 Connection ~ 5500 4400
@@
 	4800 3650 4800 3800
 $Comp
-L power:GNDD #PWR0147
+L bottom-board-rescue:GNDD-power #PWR0147
 U 1 1 5522D8E7
 P 2850 4300
@@
 $EndComp
 $Comp
-L power:GNDD #PWR0148
+L bottom-board-rescue:GNDD-power #PWR0148
 U 1 1 5522FFC1
 P 3350 3400
@@
 	-1   0    0    1
 $EndComp
-$Comp
-L power:+3.3V #PWR0149
-U 1 1 55FA5E06
-P 3350 2450
-F 0 "#PWR0149" H 3350 2300 50  0001 C CNN
-F 1 "+3.3V" H 3350 2590 50  0000 C CNN
-F 2 "" H 3350 2450 60  0000 C CNN
-F 3 "" H 3350 2450 60  0000 C CNN
-	1    3350 2450
-	1    0    0    -1
-$EndComp
-Wire Wire Line
-	3350 2450 3350 2550
-Wire Wire Line
-	3350 2950 3350 3150
+Wire Wire Line
+	3350 2950 3350 3050
 Wire Wire Line
 	3350 3350 3350 3400
@@
 Connection ~ 3350 3050
 $Comp
-L power:+3.3V #PWR0150
+L bottom-board-rescue:+3.3V-power #PWR0150
 U 1 1 55FA859A
 P 2850 3350
@@
 	2850 4250 2850 4300
 Wire Wire Line
-	2850 3850 2850 4050
+	2850 3850 2850 3950
 Wire Wire Line
 	2700 3950 2850 3950
@@
 Connection ~ 4800 4000
 $Comp
-L power:GNDD #PWR0151
+L bottom-board-rescue:GNDD-power #PWR0151
 U 1 1 55FB1C75
 P 4800 4350
@@
 	4800 4300 4800 4350
 Wire Wire Line
-	5200 2750 5550 2750
+	5200 2750 5300 2750
 Wire Wire Line
 	4800 3100 4800 3500
 Connection ~ 4800 3500
 $Comp
-L power:+3.3V #PWR0152
+L bottom-board-rescue:+3.3V-power #PWR0152
 U 1 1 55FB2896
 P 4800 2800
@@
 Wire Wire Line
 	4800 2800 4800 2900
+Wire Wire Line
+	3350 2550 3350 2450
+Wire Wire Line
+	5300 2750 5300 2900
+Wire Wire Line
+	5300 2750 5550 2750
+Wire Wire Line
+	5500 4400 5500 4450
+Wire Wire Line
+	6650 3450 6950 3450
+Wire Wire Line
+	6650 3150 6950 3150
+Wire Wire Line
+	4450 3300 4550 3300
+Wire Wire Line
+	4800 3800 4900 3800
+Wire Wire Line
+	3350 3050 3350 3150
+Wire Wire Line
+	2850 3950 2850 4050
+Wire Wire Line
+	4800 4000 4900 4000
+Wire Wire Line
+	4800 3500 4900 3500
+$Comp
+L bottom-board-rescue:+3.3V-power #PWR0149
+U 1 1 5C959C67
+P 3350 2450
+F 0 "#PWR0149" H 3350 2300 50  0001 C CNN
+F 1 "+3.3V" H 3350 2590 50  0000 C CNN
+F 2 "" H 3350 2450 60  0000 C CNN
+F 3 "" H 3350 2450 60  0000 C CNN
+	1    3350 2450
+	1    0    0    -1
+$EndComp
 $EndSCHEMATC

Commit message: updated footprints and MPN's
Parts:
- C54: footprint Capacitors_SMD:C_0603 -> Capacitor_SMD:C_0603_1608Metric
- Q14, Q15: footprint Housings_SOT-23_SOT-143_TSOT-6:SOT-23 -> Package_TO_SOT_SMD:SOT-23
- R53, R54, R55, R56, R57, R58: footprint Resistors_SMD:R_0603 -> Resistor_SMD:R_0603_1608Metric
- R59, R60, R61, R62, R63: footprint Resistors_SMD:R_0805 -> Resistor_SMD:R_0805_2012Metric
- U12: footprint Housings_SOIC:SOIC-14_3.9x8.7mm_Pitch1.27mm -> Package_SO:SOIC-14_3.9x8.7mm_P1.27mm
Changed lines of the file:
@@
 EESchema Schematic File Version 4
 LIBS:bottom-board-cache
-EELAYER 26 0
+EELAYER 29 0
 EELAYER END
 $Descr A4 11693 8268
@@
 F 0 "R63" H 6700 3350 50  0000 L CNN
 F 1 "100R" H 6700 3250 50  0000 L CNN
-F 2 "Resistors_SMD:R_0805" H 6650 3300 60  0001 C CNN
+F 2 "Resistor_SMD:R_0805_2012Metric" H 6650 3300 60  0001 C CNN
 F 3 "" H 6650 3300 60  0000 C CNN
 F 4 "ERJ-P06J101V" H 100 1000 50  0001 C CNN "MPN"
@@
 F 0 "R59" H 5900 3250 50  0000 L CNN
 F 1 "56R" H 5900 3150 50  0000 L CNN
-F 2 "Resistors_SMD:R_0805" H 6100 3200 60  0001 C CNN
+F 2 "Resistor_SMD:R_0805_2012Metric" H 6100 3200 60  0001 C CNN
 F 3 "" H 6100 3200 60  0000 C CNN
 F 4 "ERJ-P6WJ560V" H 100 1000 50  0001 C CNN "MPN"
@@
 F 0 "R60" H 6150 3450 50  0000 L CNN
 F 1 "56R" H 6150 3350 50  0000 L CNN
-F 2 "Resistors_SMD:R_0805" H 6100 3400 60  0001 C CNN
+F 2 "Resistor_SMD:R_0805_2012Metric" H 6100 3400 60  0001 C CNN
 F 3 "" H 6100 3400 60  0000 C CNN
 F 4 "ERJ-P6WJ560V" H 100 1000 50  0001 C CNN "MPN"
@@
 F 0 "C54" V 5700 2800 50  0000 L CNN
 F 1 "100nF" V 5550 2650 50  0000 L CNN
-F 2 "Capacitors_SMD:C_0603" H 5650 2750 60  0001 C CNN
+F 2 "Capacitor_SMD:C_0603_1608Metric" H 5650 2750 60  0001 C CNN
 F 3 "" H 5650 2750 60  0000 C CNN
 F 4 "C1608X7R1E104K080AA" H 800 1000 50  0001 C CNN "MPN"
@@
 F 0 "R56" V 4550 3200 50  0000 L CNN
 F 1 "100R" V 4750 3200 50  0000 L CNN
-F 2 "Resistors_SMD:R_0603" H 4650 3300 60  0001 C CNN
+F 2 "Resistor_SMD:R_0603_1608Metric" H 4650 3300 60  0001 C CNN
 F 3 "" H 4650 3300 60  0000 C CNN
 F 4 "RMCF0603JT100R" H 100 1000 50  0001 C CNN "MPN"
@@
 F 0 "R55" V 4500 3700 50  0000 L CNN
 F 1 "100R" V 4700 3700 50  0000 L CNN
-F 2 "Resistors_SMD:R_0603" H 4600 3800 60  0001 C CNN
+F 2 "Resistor_SMD:R_0603_1608Metric" H 4600 3800 60  0001 C CNN
 F 3 "" H 4600 3800 60  0000 C CNN
 F 4 "RMCF0603JT100R" H 50  1000 50  0001 C CNN "MPN"
@@
 F 0 "U12" H 5200 2950 50  0000 L CNN
 F 1 "ISL83491" H 5400 4200 50  0000 L CNN
-F 2 "Housings_SOIC:SOIC-14_3.9x8.7mm_Pitch1.27mm" H 5400 3600 50  0001 C CIN
+F 2 "Package_SO:SOIC-14_3.9x8.7mm_P1.27mm" H 5400 3600 50  0001 C CIN
 F 3 "" H 5400 3600 60  0000 C CNN
 F 4 "ISL83491IBZ" H 100 1000 50  0001 C CNN "MPN"
@@
 F 0 "R61" H 6150 3750 50  0000 L CNN
 F 1 "56R" H 6150 3650 50  0000 L CNN
-F 2 "Resistors_SMD:R_0805" H 6350 3700 60  0001 C CNN
+F 2 "Resistor_SMD:R_0805_2012Metric" H 6350 3700 60  0001 C CNN
 F 3 "" H 6350 3700 60  0000 C CNN
 F 4 "ERJ-P6WJ560V" H 100 1000 50  0001 C CNN "MPN"
@@
 F 0 "R62" H 6400 3950 50  0000 L CNN
 F 1 "56R" H 6400 3850 50  0000 L CNN
-F 2 "Resistors_SMD:R_0805" H 6350 3900 60  0001 C CNN
+F 2 "Resistor_SMD:R_0805_2012Metric" H 6350 3900 60  0001 C CNN
 F 3 "" H 6350 3900 60  0000 C CNN
 F 4 "ERJ-P6WJ560V" H 100 1000 50  0001 C CNN "MPN"
@@
 F 0 "R54" H 3400 3300 50  0000 L CNN
 F 1 "10k" H 3400 3200 50  0000 L CNN
-F 2 "Resistors_SMD:R_0603" H 3350 3250 60  0001 C CNN
+F 2 "Resistor_SMD:R_0603_1608Metric" H 3350 3250 60  0001 C CNN
 F 3 "" H 3350 3250 60  0000 C CNN
 F 4 "RMCF0603JT10K0" H 100 1950 50  0001 C CNN "MPN"
@@
 F 0 "R53" H 2900 4200 50  0000 L CNN
 F 1 "10k" H 2900 4100 50  0000 L CNN
-F 2 "Resistors_SMD:R_0603" H 2850 4150 60  0001 C CNN
+F 2 "Resistor_SMD:R_0603_1608Metric" H 2850 4150 60  0001 C CNN
 F 3 "" H 2850 4150 60  0000 C CNN
 F 4 "RMCF0603JT10K0" H -400 1350 50  0001 C CNN "MPN"
@@
 F 0 "Q15" H 3750 2800 50  0000 R CNN
 F 1 "BSS84" H 3850 2700 50  0000 R CNN
-F 2 "Housings_SOT-23_SOT-143_TSOT-6:SOT-23" H 3650 2850 29  0001 C CNN
+F 2 "Package_TO_SOT_SMD:SOT-23" H 3650 2850 29  0001 C CNN
 F 3 "" H 3450 2750 60  0000 C CNN
 F 4 "BSS84" H 3450 2750 60  0001 C CNN "MPN"
@@
 F 0 "Q14" H 3250 3700 50  0000 R CNN
 F 1 "BSS84" H 3350 3600 50  0000 R CNN
-F 2 "Housings_SOT-23_SOT-143_TSOT-6:SOT-23" H 3150 3750 29  0001 C CNN
+F 2 "Package_TO_SOT_SMD:SOT-23" H 3150 3750 29  0001 C CNN
 F 3 "" H 2950 3650 60  0000 C CNN
 F 4 "BSS84" H 2950 3650 60  0001 C CNN "MPN"
@@
 F 0 "R57" H 4850 3050 50  0000 L CNN
 F 1 "10k" H 4850 2950 50  0000 L CNN
-F 2 "Resistors_SMD:R_0603" H 4800 3000 60  0001 C CNN
+F 2 "Resistor_SMD:R_0603_1608Metric" H 4800 3000 60  0001 C CNN
 F 3 "" H 4800 3000 60  0000 C CNN
 F 4 "RMCF0603JT10K0" H 1550 1700 50  0001 C CNN "MPN"
@@
 F 0 "R58" H 4850 4250 50  0000 L CNN
 F 1 "10k" H 4850 4150 50  0000 L CNN
-F 2 "Resistors_SMD:R_0603" H 4800 4200 60  0001 C CNN
+F 2 "Resistor_SMD:R_0603_1608Metric" H 4800 4200 60  0001 C CNN
 F 3 "" H 4800 4200 60  0000 C CNN
 F 4 "RMCF0603JT10K0" H 1550 2900 50  0001 C CNN "MPN"
