File: hw-design/bottom-board/coreboard.sch (KiCad schematic (older format))
At the start: 12 parts, among them SW1 SW_PUSH, U4 AT24CS08-STUM, U5 Core_AW204x

Commit message: Changed SODIM to Marsboard header + added liniar regulator for audio codec
Parts:
- removed R3: 10k, Resistors_SMD:R_0603, symbol bottom-board-rescue:R_Small
- removed U5: Core_AW204x, footprints:Socket_SODIMM_DDR3_TE_2013289, symbol itead:Core_AW204x
- added J7, J8: Conn_02x50_Odd_Even, footprints-local:Pin_Header_Straight_2x50_Pitch1.27mm_SMD, symbol bottom-board-rescue:Conn_02x50_Odd_Even-header
- U4: footprint Housings_SOT-23_SOT-143_TSOT-6:SOT-23-5 -> Package_TO_SOT_SMD:SOT-23-5
Connections:
- net labels removed: SD0_CLK, SD0_CMD, SD0_D0, SD0_D1, SD0_D2, SD0_D3, SD0_DETECT
- wire segments 138 -> 141
- no-connect marks 129 -> 130
Other:
- moved on the sheet: C30, C31, C58, C59, R15, R16

Commit message: updated footprints and MPN's
Parts:
- C30, C58: footprint Capacitors_SMD:C_0805 -> Capacitor_SMD:C_0805_2012Metric
- C31, C59, C60: footprint Capacitors_SMD:C_0603 -> Capacitor_SMD:C_0603_1608Metric
- J7, J8: footprint footprints-local:Pin_Header_Straight_2x50_Pitch1.27mm_SMD -> footprints:Pin_Header_Straight_2x50_Pitch1.27mm_SMD
- R14, R15, R16: footprint Resistors_SMD:R_0603 -> Resistor_SMD:R_0603_1608Metric
Changed lines of the file:
@@
 EESchema Schematic File Version 4
 LIBS:bottom-board-cache
-EELAYER 26 0
+EELAYER 29 0
 EELAYER END
 $Descr A4 11693 8268
@@
 F 0 "C31" V 2250 4200 50  0000 L CNN
 F 1 "100nF" V 2150 4200 50  0000 L CNN
-F 2 "Capacitors_SMD:C_0603" H 2200 4150 60  0001 C CNN
+F 2 "Capacitor_SMD:C_0603_1608Metric" H 2200 4150 60  0001 C CNN
 F 3 "" H 2200 4150 60  0000 C CNN
 F 4 "C1608X7R1E104K080AA" H -8700 2050 50  0001 C CNN "MPN"
@@
 F 0 "R14" H 1800 6250 50  0000 L CNN
 F 1 "10k" H 1800 6150 50  0000 L CNN
-F 2 "Resistors_SMD:R_0603" H 1750 6200 60  0001 C CNN
+F 2 "Resistor_SMD:R_0603_1608Metric" H 1750 6200 60  0001 C CNN
 F 3 "" H 1750 6200 60  0000 C CNN
 F 4 "RMCF0603JT10K0" H 0   -450 50  0001 C CNN "MPN"
@@
 F 0 "C30" V 2250 4000 50  0000 L CNN
 F 1 "10uF" V 2150 4000 50  0000 L CNN
-F 2 "Capacitors_SMD:C_0805" H 2200 3950 60  0001 C CNN
+F 2 "Capacitor_SMD:C_0805_2012Metric" H 2200 3950 60  0001 C CNN
 F 3 "" H 2200 3950 60  0000 C CNN
 F 4 "GRM219R61E106KA12D" H -3100 -1400 50  0001 C CNN "MPN"
@@
 F 0 "R16" V 4450 2950 50  0000 L CNN
 F 1 "2k7" V 4550 2940 50  0000 L CNN
-F 2 "Resistors_SMD:R_0603" H 4550 3000 60  0001 C CNN
+F 2 "Resistor_SMD:R_0603_1608Metric" H 4550 3000 60  0001 C CNN
 F 3 "" H 4550 3000 60  0000 C CNN
 F 4 "RMCF0603JT2K70" H -4000 1150 50  0001 C CNN "MPN"
@@
 F 0 "R15" V 4650 4500 50  0000 L CNN
 F 1 "2k7" V 4550 4490 50  0000 L CNN
-F 2 "Resistors_SMD:R_0603" H 4550 4550 60  0001 C CNN
+F 2 "Resistor_SMD:R_0603_1608Metric" H 4550 4550 60  0001 C CNN
 F 3 "" H 4550 4550 60  0000 C CNN
 F 4 "RMCF0603JT2K70" H -3900 2700 50  0001 C CNN "MPN"
@@
 F 0 "C59" V 2850 950 50  0000 L CNN
 F 1 "100nF" V 2750 950 50  0000 L CNN
-F 2 "Capacitors_SMD:C_0603" H 2800 900 60  0001 C CNN
+F 2 "Capacitor_SMD:C_0603_1608Metric" H 2800 900 60  0001 C CNN
 F 3 "" H 2800 900 60  0000 C CNN
 F 4 "C1608X7R1E104K080AA" H -8100 -1200 50  0001 C CNN "MPN"
@@
 F 0 "C58" V 3050 950 50  0000 L CNN
 F 1 "10uF" V 2950 950 50  0000 L CNN
-F 2 "Capacitors_SMD:C_0805" H 3000 900 60  0001 C CNN
+F 2 "Capacitor_SMD:C_0805_2012Metric" H 3000 900 60  0001 C CNN
 F 3 "" H 3000 900 60  0000 C CNN
 F 4 "GRM219R61E106KA12D" H -2300 -4450 50  0001 C CNN "MPN"
@@
 F 0 "C60" V 5900 6400 50  0000 L CNN
 F 1 "100nF" V 5800 6400 50  0000 L CNN
-F 2 "Capacitors_SMD:C_0603" H 5850 6350 60  0001 C CNN
+F 2 "Capacitor_SMD:C_0603_1608Metric" H 5850 6350 60  0001 C CNN
 F 3 "" H 5850 6350 60  0000 C CNN
 F 4 "C1608X7R1E104K080AA" H -5050 4250 50  0001 C CNN "MPN"
@@
 F 0 "J7" V 5446 4279 50  0000 L CNN
 F 1 "Conn_02x50_Odd_Even" H 4900 -850 50  0000 L CNN
-F 2 "footprints-local:Pin_Header_Straight_2x50_Pitch1.27mm_SMD" H 5350 2300 50  0001 C CNN
+F 2 "footprints:Pin_Header_Straight_2x50_Pitch1.27mm_SMD" H 5350 2300 50  0001 C CNN
 F 3 "~" H 5350 2300 50  0001 C CNN
 	1    5400 1800
@@
 F 0 "J8" V 5296 6329 50  0000 L CNN
 F 1 "Conn_02x50_Odd_Even" H 4800 1250 50  0000 L CNN
-F 2 "footprints-local:Pin_Header_Straight_2x50_Pitch1.27mm_SMD" H 5200 4350 50  0001 C CNN
+F 2 "footprints:Pin_Header_Straight_2x50_Pitch1.27mm_SMD" H 5200 4350 50  0001 C CNN
 F 3 "~" H 5200 4350 50  0001 C CNN
 	1    5250 3850
