File: hw-design/bottom-board/mechanics.sch (KiCad schematic (older format))
At the start: 9 parts

Commit message: Changed SODIM to Marsboard header + added liniar regulator for audio codec
Parts:
- removed H6: Standoff, footprints:9774027151R, symbol local-components:HOLE
- FID1, FID2, FID3: symbol local-components:FIDUCIAL -> bottom-board-rescue:FIDUCIAL-local-components
- H1, H2, H3, H4, H5: symbol local-components:HOLE -> bottom-board-rescue:HOLE-local-components
Changed lines of the file:
@@
 $EndDescr
 $Comp
-L local-components:FIDUCIAL FID1
+L bottom-board-rescue:FIDUCIAL-local-components FID1
 U 1 1 55FC074E
 P 1400 1400
+AR Path="/55FC074E" Ref="FID1"  Part="1"
+AR Path="/55FC02AF/55FC074E" Ref="FID1"  Part="1"
 F 0 "FID1" H 1400 1125 50  0000 C CNN
 F 1 "FIDUCIAL" H 1400 1675 50  0000 C CNN
@@
 $EndComp
 $Comp
-L local-components:HOLE H1
+L bottom-board-rescue:HOLE-local-components H1
 U 1 1 55FC0943
 P 3350 1400
+AR Path="/55FC0943" Ref="H1"  Part="1"
+AR Path="/55FC02AF/55FC0943" Ref="H1"  Part="1"
 F 0 "H1" H 3350 1220 50  0000 C CNN
 F 1 "HOLE" H 3350 1570 50  0000 C CNN
@@
 $EndComp
 $Comp
-L local-components:FIDUCIAL FID2
+L bottom-board-rescue:FIDUCIAL-local-components FID2
 U 1 1 55FC1F87
 P 1900 1400
+AR Path="/55FC1F87" Ref="FID2"  Part="1"
+AR Path="/55FC02AF/55FC1F87" Ref="FID2"  Part="1"
 F 0 "FID2" H 1900 1125 50  0000 C CNN
 F 1 "FIDUCIAL" H 1900 1675 50  0000 C CNN
@@
 $EndComp
 $Comp
-L local-components:FIDUCIAL FID3
+L bottom-board-rescue:FIDUCIAL-local-components FID3
 U 1 1 55FC1FBF
 P 2400 1400
+AR Path="/55FC1FBF" Ref="FID3"  Part="1"
+AR Path="/55FC02AF/55FC1FBF" Ref="FID3"  Part="1"
 F 0 "FID3" H 2400 1125 50  0000 C CNN
 F 1 "FIDUCIAL" H 2400 1675 50  0000 C CNN
@@
 $EndComp
 $Comp
-L local-components:HOLE H2
+L bottom-board-rescue:HOLE-local-components H2
 U 1 1 55FC2212
 P 3700 1400
+AR Path="/55FC2212" Ref="H2"  Part="1"
+AR Path="/55FC02AF/55FC2212" Ref="H2"  Part="1"
 F 0 "H2" H 3700 1220 50  0000 C CNN
 F 1 "HOLE" H 3700 1570 50  0000 C CNN
@@
 $EndComp
 $Comp
-L local-components:HOLE H3
+L bottom-board-rescue:HOLE-local-components H3
 U 1 1 55FC224E
 P 4050 1400
+AR Path="/55FC224E" Ref="H3"  Part="1"
+AR Path="/55FC02AF/55FC224E" Ref="H3"  Part="1"
 F 0 "H3" H 4050 1220 50  0000 C CNN
 F 1 "HOLE" H 4050 1570 50  0000 C CNN
@@
 $EndComp
 $Comp
-L local-components:HOLE H4
+L bottom-board-rescue:HOLE-local-components H4
 U 1 1 55FC227A
 P 4400 1400
+AR Path="/55FC227A" Ref="H4"  Part="1"
+AR Path="/55FC02AF/55FC227A" Ref="H4"  Part="1"
 F 0 "H4" H 4400 1220 50  0000 C CNN
 F 1 "HOLE" H 4400 1570 50  0000 C CNN
@@
 $EndComp
 $Comp
-L local-components:HOLE H5
+L bottom-board-rescue:HOLE-local-components H5
 U 1 1 55FC22B0
 P 4750 1400
+AR Path="/55FC22B0" Ref="H5"  Part="1"
+AR Path="/55FC02AF/55FC22B0" Ref="H5"  Part="1"
 F 0 "H5" H 4750 1220 50  0000 C CNN
 F 1 "HOLE" H 4750 1570 50  0000 C CNN
@@
 	1    0    0    -1
 $EndComp
-$Comp
-L local-components:HOLE H6
-U 1 1 55FBDF5C
-P 5450 1400
-F 0 "H6" H 5450 1220 50  0000 C CNN
-F 1 "Standoff" H 5450 1570 50  0000 C CNN
-F 2 "footprints:9774027151R" H 5450 1400 60  0001 C CNN
-F 3 "" H 5450 1400 60  0000 C CNN
-F 4 "9774027151R" H 5450 1400 60  0001 C CNN "MPN"
-	1    5450 1400
-	1    0    0    -1
-$EndComp
