File: hw-design/bottom-board/audio-codec.sch (KiCad schematic (older format))
At the start: 33 parts, among them U3 CS4245

Commit message: Changed SODIM to Marsboard header + added liniar regulator for audio codec
Parts:
- removed C25: 10uF, Capacitors_SMD:c_elec_5x5.3, symbol bottom-board-rescue:CP_Small
- removed R11: 10k, Resistors_SMD:R_0603, symbol bottom-board-rescue:R_Small
- removed U3: CS4245, Housings_QFP:LQFP-48_7x7mm_Pitch0.5mm, symbol bottom-board-rescue:CS4245
- added C25: 10uF, Capacitor_SMD:C_0805_2012Metric, symbol bottom-board-rescue:C_Small
- added C37: 100nF, Capacitor_SMD:C_0402_1005Metric, symbol bottom-board-rescue:C_Small
- added C62: 10uF, Capacitor_SMD:CP_Elec_5x5.3, symbol bottom-board-rescue:CP_Small
- added R17: 10k, Resistor_SMD:R_0201_0603Metric, symbol bottom-board-rescue:R_Small
- added R3: 22R, Resistors_SMD:R_0603, symbol bottom-board-rescue:R_Small
- added R4: 22R, Resistor_SMD:R_0603_1608Metric_Pad1.05x0.95mm_HandSolder, symbol bottom-board-rescue:R_Small
- added U13: AP2120N-3.3, Package_TO_SOT_SMD:SOT-23, symbol bottom-board-rescue:AP2120N-3.3-local-components2
- added U3: CS4245, Package_QFP:LQFP-48_7x7mm_P0.5mm, symbol bottom-board-rescue:CS4245-Audio
- C24: value 100nF -> 1uF; footprint Capacitors_SMD:C_0402 -> Capacitor_SMD:C_0805_2012Metric; MPN C1005X7R1E104K050BB -> C2012X7R1E105K125AB
- R10, R9: value 100R -> 22R
Connections:
- net labels added: +3.3VA
- net labels removed: +3.3V
- wire segments 127 -> 176
Other:
- moved on the sheet: C12, C13, C14, C15, C16, C17, C18, C19, C20, C21, C22, C23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

Commit message: updated footprints and MPN's
Parts:
- C12, C15, C18, C19, C20: footprint Capacitors_SMD:C_0805 -> Capacitor_SMD:C_0805_2012Metric
- C13, C14, C16, C17, C21, C22, C26, C28: footprint Capacitors_SMD:C_0402 -> Capacitor_SMD:C_0402_1005Metric
- C23: footprint Capacitors_SMD:c_elec_5x5.3 -> Capacitor_SMD:CP_Elec_6.3x5.3
- C25: MPN C2012X7R1E105K125AB -> GRM219R61E106KA12D
- C27, C29: footprint Capacitors_SMD:c_elec_6.3x5.3 -> Capacitor_SMD:CP_Elec_6.3x5.3
- C62: footprint Capacitor_SMD:CP_Elec_5x5.3 -> Capacitor_SMD:CP_Elec_6.3x5.3
- CA1, CA2: footprint Capacitors_SMD:C_0603 -> Capacitor_SMD:C_0603_1608Metric
- D3, D4: footprint Housings_SOT-23_SOT-143_TSOT-6:SOT-23 -> Package_TO_SOT_SMD:SOT-23
- R1, R10, R12, R13, R2, R3, R5, R6, R7, R9: footprint Resistors_SMD:R_0603 -> Resistor_SMD:R_0603_1608Metric
- R17: footprint Resistor_SMD:R_0201_0603Metric -> Resistor_SMD:R_0603_1608Metric
- R4: footprint Resistor_SMD:R_0603_1608Metric_Pad1.05x0.95mm_HandSolder -> Resistor_SMD:R_0603_1608Metric

Commit message: correct tracks that overlap with new footprints
Parts:
- R10, R9: MPN RMCF0603JT100R -> RMCF0603JT22R0
Changed lines of the file:
@@
 F 2 "Resistor_SMD:R_0603_1608Metric" H 4450 3950 60  0001 C CNN
 F 3 "" H 4450 3950 60  0000 C CNN
-F 4 "RMCF0603JT100R" H 150 1600 50  0001 C CNN "MPN"
+F 4 "RMCF0603JT22R0" H 150 1600 50  0001 C CNN "MPN"
 	1    4450 3950
 	0    1    1    0
@@
 F 2 "Resistor_SMD:R_0603_1608Metric" H 4450 4050 60  0001 C CNN
 F 3 "" H 4450 4050 60  0000 C CNN
-F 4 "RMCF0603JT100R" H 150 1600 50  0001 C CNN "MPN"
+F 4 "RMCF0603JT22R0" H 150 1600 50  0001 C CNN "MPN"
 	1    4450 4050
 	0    1    1    0
