File: hw-design/bottom-board/audio-inputs.sch (KiCad schematic (older format))
At the start: 56 parts, among them Q1 2N7002, Q2 2N7002, Q3 J112, Q4 J112, Q5 J112, Q6 J112, Q7 2N7002, Q8 2N7002, U6 LM4562

Commit message: Changed SODIM to Marsboard header + added liniar regulator for audio codec
Connections:
- wire segments 128 -> 172

Commit message: updated footprints and MPN's
Parts:
- C34, CA10, CA9: footprint Capacitors_SMD:c_elec_5x5.3 -> Capacitor_SMD:CP_Elec_5x5.3
- C35, CA3, CA4, CA7, CA8: footprint Capacitors_SMD:C_0603 -> Capacitor_SMD:C_0603_1608Metric
- C38: footprint Capacitors_SMD:c_elec_6.3x5.3 -> Capacitor_SMD:CP_Elec_6.3x5.3
- CA5, CA6: footprint Capacitors_SMD:C_1206 -> Capacitor_SMD:C_1206_3216Metric
- D10, D5, D6, D9: footprint Diodes_SMD:SOD-323 -> Diode_SMD:D_SOD-323
- D7, D8, Q1, Q2, Q3, Q4, Q5, Q6, Q7, Q8: footprint Housings_SOT-23_SOT-143_TSOT-6:SOT-23 -> Package_TO_SOT_SMD:SOT-23
- R20, R21, R22, R23, R24, R25, R26, R27, R28, R29, R30, R31, RA1, RA10, RA11, RA12, RA13, RA14, RA15, RA17, RA18, RA2, RA3, RA4, RA5, RA6, RA7, RA8, RA9: footprint Resistors_SMD:R_0603 -> Resistor_SMD:R_0603_1608Metric
- U6: footprint Housings_SOIC:SOIC-8_3.9x4.9mm_Pitch1.27mm -> Package_SO:SOIC-8-1EP_3.9x4.9mm_P1.27mm_EP2.41x3.81mm_ThermalVias

Commit message: correct tracks that overlap with new footprints
Parts:
- RA16: footprint Resistors_SMD:R_0603 -> Resistor_SMD:R_0603_1608Metric
- U6: footprint Package_SO:SOIC-8-1EP_3.9x4.9mm_P1.27mm_EP2.41x3.81mm_ThermalVias -> Package_SO:SOIC-8_3.9x4.9mm_P1.27mm
Changed lines of the file:
@@
 F 0 "U6" H 4050 5300 60  0001 L CNN
 F 1 "LM4562" H 4050 5000 60  0000 L CNN
-F 2 "Package_SO:SOIC-8-1EP_3.9x4.9mm_P1.27mm_EP2.41x3.81mm_ThermalVias" H 4050 5150 60  0001 C CNN
+F 2 "Package_SO:SOIC-8_3.9x4.9mm_P1.27mm" H 4050 5150 60  0001 C CNN
 F 3 "" H 4050 5150 60  0000 C CNN
 F 4 "LM4562MAX/NOPB" H 50  3650 50  0001 C CNN "MPN"
@@
 F 0 "RA16" V 4600 5050 50  0000 L CNN
 F 1 "100R" V 4800 5050 50  0000 L CNN
-F 2 "Resistors_SMD:R_0603" H 4700 5150 60  0001 C CNN
+F 2 "Resistor_SMD:R_0603_1608Metric" H 4700 5150 60  0001 C CNN
 F 3 "" H 4700 5150 60  0000 C CNN
 F 4 "ERA-3AEB101V" H -5100 2400 50  0001 C CNN "MPN"
@@
 F 0 "U6" H 4000 1650 60  0000 L CNN
 F 1 "LM4562" H 4000 1350 60  0000 L CNN
-F 2 "Package_SO:SOIC-8-1EP_3.9x4.9mm_P1.27mm_EP2.41x3.81mm_ThermalVias" H 4000 1500 60  0001 C CNN
+F 2 "Package_SO:SOIC-8_3.9x4.9mm_P1.27mm" H 4000 1500 60  0001 C CNN
 F 3 "" H 4000 1500 60  0000 C CNN
 F 4 "LM4562MAX/NOPB" H -5150 -1250 50  0001 C CNN "MPN"
