File: hw-design/bottom-board/audio-outputs.sch (KiCad schematic (older format))
At the start: 49 parts, among them K1 IM06TS, K2 IM06TS, Q10 2N7002, Q9 2N7002, U7 LM4562, U8 LM4562

Commit message: Changed SODIM to Marsboard header + added liniar regulator for audio codec
Connections:
- wire segments 149 -> 190

Commit message: Changed capacitor posistion & changed relay footprint
Parts:
- K1, K2: footprint footprints:Relay_DPDT_IMXXTS -> footprints:Relay_DPDT_Omron_G6S-2F-good_pinout
Changed lines of the file:
@@
 F 0 "K1" H 8200 2500 50  0000 L CNN
 F 1 "IM06TS" H 8200 2400 50  0000 L CNN
-F 2 "footprints:Relay_DPDT_IMXXTS" H 7350 2350 60  0001 C CNN
+F 2 "footprints:Relay_DPDT_Omron_G6S-2F-good_pinout" H 7350 2350 60  0001 C CNN
 F 3 "" H 7350 2350 60  0000 C CNN
 F 4 "IM06TS" H 7350 2350 60  0001 C CNN "MPN"
@@
 F 0 "K2" H 8200 5350 50  0000 L CNN
 F 1 "IM06TS" H 8200 5250 50  0000 L CNN
-F 2 "footprints:Relay_DPDT_IMXXTS" H 7350 5200 60  0001 C CNN
+F 2 "footprints:Relay_DPDT_Omron_G6S-2F-good_pinout" H 7350 5200 60  0001 C CNN
 F 3 "" H 7350 5200 60  0000 C CNN
 F 4 "IM06TS" H 7350 5200 60  0001 C CNN "MPN"

Commit message: updated footprints and MPN's
Parts:
- C39: footprint Capacitors_SMD:c_elec_6.3x5.3 -> Capacitor_SMD:CP_Elec_6.3x5.3
- C40, C41, CA11, CA12, CA17, CA18: footprint Capacitors_SMD:c_elec_5x5.3 -> Capacitor_SMD:CP_Elec_5x5.3
- C42, C43, C44, C45, CA13, CA14, CA15, CA16: footprint Capacitors_SMD:C_0603 -> Capacitor_SMD:C_0603_1608Metric
- CA19, CA20: footprint Capacitors_SMD:c_elec_6.3x7.7 -> Capacitor_SMD:CP_Elec_6.3x7.7
- D11, D12: footprint Diodes_SMD:SOD-323 -> Diode_SMD:D_SOD-323
- Q10, Q9: footprint Housings_SOT-23_SOT-143_TSOT-6:SOT-23 -> Package_TO_SOT_SMD:SOT-23
- R34, R35, R36, R37, RA19, RA20, RA21, RA22, RA23, RA24, RA25, RA26, RA27, RA28, RA29, RA30, RA31, RA32, RA33, RA34, RA35, RA36, RA37, RA38: footprint Resistors_SMD:R_0603 -> Resistor_SMD:R_0603_1608Metric
- U7, U8: footprint Housings_SOIC:SOIC-8_3.9x4.9mm_Pitch1.27mm -> Package_SO:SOIC-8-1EP_3.9x4.9mm_P1.27mm_EP2.41x3.81mm_ThermalVias

Commit message: correct tracks that overlap with new footprints
Parts:
- U7, U8: footprint Package_SO:SOIC-8-1EP_3.9x4.9mm_P1.27mm_EP2.41x3.81mm_ThermalVias -> Package_SO:SOIC-8_3.9x4.9mm_P1.27mm
Changed lines of the file:
@@
 F 0 "U7" H 2950 1800 60  0000 L CNN
 F 1 "LM4562" H 3350 1450 60  0000 L CNN
-F 2 "Package_SO:SOIC-8-1EP_3.9x4.9mm_P1.27mm_EP2.41x3.81mm_ThermalVias" H 3300 1550 60  0001 C CNN
+F 2 "Package_SO:SOIC-8_3.9x4.9mm_P1.27mm" H 3300 1550 60  0001 C CNN
 F 3 "" H 3300 1550 60  0000 C CNN
 F 4 "LM4562MAX/NOPB" H 0   0   50  0001 C CNN "MPN"
@@
 F 0 "U8" H 2950 4650 60  0000 L CNN
 F 1 "LM4562" H 3350 4300 60  0000 L CNN
-F 2 "Package_SO:SOIC-8-1EP_3.9x4.9mm_P1.27mm_EP2.41x3.81mm_ThermalVias" H 3300 4400 60  0001 C CNN
+F 2 "Package_SO:SOIC-8_3.9x4.9mm_P1.27mm" H 3300 4400 60  0001 C CNN
 F 3 "" H 3300 4400 60  0000 C CNN
 F 4 "LM4562MAX/NOPB" H -1400 2750 50  0001 C CNN "MPN"
@@
 F 0 "U7" H 4350 1900 60  0000 L CNN
 F 1 "LM4562" H 4750 1550 60  0000 L CNN
-F 2 "Package_SO:SOIC-8-1EP_3.9x4.9mm_P1.27mm_EP2.41x3.81mm_ThermalVias" H 4700 1650 60  0001 C CNN
+F 2 "Package_SO:SOIC-8_3.9x4.9mm_P1.27mm" H 4700 1650 60  0001 C CNN
 F 3 "" H 4700 1650 60  0000 C CNN
 F 4 "LM4562MAX/NOPB" H 1400 -2800 50  0001 C CNN "MPN"
@@
 F 0 "U8" H 4350 4750 60  0000 L CNN
 F 1 "LM4562" H 4750 4400 60  0000 L CNN
-F 2 "Package_SO:SOIC-8-1EP_3.9x4.9mm_P1.27mm_EP2.41x3.81mm_ThermalVias" H 4700 4500 60  0001 C CNN
+F 2 "Package_SO:SOIC-8_3.9x4.9mm_P1.27mm" H 4700 4500 60  0001 C CNN
 F 3 "" H 4700 4500 60  0000 C CNN
 F 4 "LM4562MAX/NOPB" H 0   -50 50  0001 C CNN "MPN"
