File: hw-design/bottom-board/midi.sch (KiCad schematic (older format))
At the start: 14 parts, among them P3 DIN_5, P4 DIN_5, Q12 2N7002, Q13 2N7002, U11 6N137S

Commit message: Changed SODIM to Marsboard header + added liniar regulator for audio codec
Changed lines of the file:
@@
 $EndComp
 $Comp
-L power:GNDD #PWR0134
+L bottom-board-rescue:GNDD-power #PWR0184
 U 1 1 550D1DBB
 P 4100 3950
-F 0 "#PWR0134" H 4100 3700 50  0001 C CNN
+F 0 "#PWR0184" H 4100 3700 50  0001 C CNN
 F 1 "GNDD" H 4100 3800 50  0000 C CNN
 F 2 "" H 4100 3950 60  0000 C CNN
@@
 $EndComp
 $Comp
-L power:GNDD #PWR0135
+L bottom-board-rescue:GNDD-power #PWR0185
 U 1 1 550D24C3
 P 7050 3850
-F 0 "#PWR0135" H 7050 3600 50  0001 C CNN
+F 0 "#PWR0185" H 7050 3600 50  0001 C CNN
 F 1 "GNDD" H 7050 3700 50  0000 C CNN
 F 2 "" H 7050 3850 60  0000 C CNN
@@
 $EndComp
 $Comp
-L power:GNDD #PWR0136
+L bottom-board-rescue:GNDD-power #PWR0186
 U 1 1 550D24EA
 P 7950 4150
-F 0 "#PWR0136" H 7950 3900 50  0001 C CNN
+F 0 "#PWR0186" H 7950 3900 50  0001 C CNN
 F 1 "GNDD" H 7950 4000 50  0000 C CNN
 F 2 "" H 7950 4150 60  0000 C CNN
@@
 $EndComp
 $Comp
-L power:GNDD #PWR0137
+L bottom-board-rescue:GNDD-power #PWR0187
 U 1 1 550D2511
 P 8500 4450
-F 0 "#PWR0137" H 8500 4200 50  0001 C CNN
+F 0 "#PWR0187" H 8500 4200 50  0001 C CNN
 F 1 "GNDD" H 8500 4300 50  0000 C CNN
 F 2 "" H 8500 4450 60  0000 C CNN
@@
 $EndComp
 $Comp
-L power:+5V #PWR0138
+L bottom-board-rescue:+5V-power #PWR0188
 U 1 1 550D422C
 P 4100 3100
-F 0 "#PWR0138" H 4100 2950 50  0001 C CNN
+F 0 "#PWR0188" H 4100 2950 50  0001 C CNN
 F 1 "+5V" H 4100 3240 50  0000 C CNN
 F 2 "" H 4100 3100 60  0000 C CNN
@@
 $EndComp
 $Comp
-L power:+5V #PWR0139
+L bottom-board-rescue:+5V-power #PWR0189
 U 1 1 550D42BC
 P 6500 3200
-F 0 "#PWR0139" H 6500 3050 50  0001 C CNN
+F 0 "#PWR0189" H 6500 3050 50  0001 C CNN
 F 1 "+5V" H 6500 3340 50  0000 C CNN
 F 2 "" H 6500 3200 60  0000 C CNN
@@
 $EndComp
 $Comp
-L power:+5V #PWR0140
+L bottom-board-rescue:+5V-power #PWR0190
 U 1 1 550D4337
 P 7950 3200
-F 0 "#PWR0140" H 7950 3050 50  0001 C CNN
+F 0 "#PWR0190" H 7950 3050 50  0001 C CNN
 F 1 "+5V" H 7950 3340 50  0000 C CNN
 F 2 "" H 7950 3200 60  0000 C CNN
@@
 $EndComp
 $Comp
-L power:+5V #PWR0141
+L bottom-board-rescue:+5V-power #PWR0191
 U 1 1 550D435E
 P 8500 3450
-F 0 "#PWR0141" H 8500 3300 50  0001 C CNN
+F 0 "#PWR0191" H 8500 3300 50  0001 C CNN
 F 1 "+5V" H 8500 3590 50  0000 C CNN
 F 2 "" H 8500 3450 60  0000 C CNN
@@
 $EndComp
 $Comp
-L power:+3.3V #PWR0142
+L bottom-board-rescue:+3.3V-power #PWR0192
 U 1 1 55093BE7
 P 4500 3400
-F 0 "#PWR0142" H 4500 3250 50  0001 C CNN
+F 0 "#PWR0192" H 4500 3250 50  0001 C CNN
 F 1 "+3.3V" H 4500 3540 50  0000 C CNN
 F 2 "" H 4500 3400 60  0000 C CNN
@@
 $EndComp
 $Comp
-L power:GNDD #PWR0143
+L bottom-board-rescue:GNDD-power #PWR0193
 U 1 1 5518B6A5
 P 3700 3200
-F 0 "#PWR0143" H 3700 2950 50  0001 C CNN
+F 0 "#PWR0193" H 3700 2950 50  0001 C CNN
 F 1 "GNDD" H 3700 3050 50  0000 C CNN
 F 2 "" H 3700 3200 60  0000 C CNN

Commit message: updated footprints and MPN's
Parts:
- C53: footprint Capacitors_SMD:C_0603 -> Capacitor_SMD:C_0603_1608Metric
- R47, R49, R50: footprint Resistors_SMD:R_0805 -> Resistor_SMD:R_0805_2012Metric
- R48, R51, R52: footprint Resistors_SMD:R_0603 -> Resistor_SMD:R_0603_1608Metric
Changed lines of the file:
@@
 EESchema Schematic File Version 4
 LIBS:bottom-board-cache
-EELAYER 26 0
+EELAYER 29 0
 EELAYER END
 $Descr A4 11693 8268
@@
 F 0 "R47" H 2900 3600 50  0000 L CNN
 F 1 "220R" H 2900 3500 50  0000 L CNN
-F 2 "Resistors_SMD:R_0805" H 2850 3550 60  0001 C CNN
+F 2 "Resistor_SMD:R_0805_2012Metric" H 2850 3550 60  0001 C CNN
 F 3 "" H 2850 3550 60  0000 C CNN
 F 4 "ERJ-P06J221V" H 100 0   50  0001 C CNN "MPN"
@@
 F 0 "R49" H 6550 3400 50  0000 L CNN
 F 1 "220R" H 6550 3300 50  0000 L CNN
-F 2 "Resistors_SMD:R_0805" H 6500 3350 60  0001 C CNN
+F 2 "Resistor_SMD:R_0805_2012Metric" H 6500 3350 60  0001 C CNN
 F 3 "" H 6500 3350 60  0000 C CNN
 F 4 "ERJ-P06J221V" H 200 0   50  0001 C CNN "MPN"
@@
 F 0 "R50" H 7750 3600 50  0000 L CNN
 F 1 "220R" H 7750 3500 50  0000 L CNN
-F 2 "Resistors_SMD:R_0805" H 7700 3550 60  0001 C CNN
+F 2 "Resistor_SMD:R_0805_2012Metric" H 7700 3550 60  0001 C CNN
 F 3 "" H 7700 3550 60  0000 C CNN
 F 4 "ERJ-P06J221V" H 350 0   50  0001 C CNN "MPN"
@@
 F 0 "R51" H 8000 3400 50  0000 L CNN
 F 1 "10k" H 8000 3300 50  0000 L CNN
-F 2 "Resistors_SMD:R_0603" H 7950 3350 60  0001 C CNN
+F 2 "Resistor_SMD:R_0603_1608Metric" H 7950 3350 60  0001 C CNN
 F 3 "" H 7950 3350 60  0000 C CNN
 F 4 "RMCF0603JT10K0" H 350 0   50  0001 C CNN "MPN"
@@
 F 0 "R52" H 8550 3700 50  0000 L CNN
 F 1 "10k" H 8550 3600 50  0000 L CNN
-F 2 "Resistors_SMD:R_0603" H 8500 3650 60  0001 C CNN
+F 2 "Resistor_SMD:R_0603_1608Metric" H 8500 3650 60  0001 C CNN
 F 3 "" H 8500 3650 60  0000 C CNN
 F 4 "RMCF0603JT10K0" H 150 0   50  0001 C CNN "MPN"
@@
 F 0 "R48" H 4550 3600 50  0000 L CNN
 F 1 "10k" H 4550 3500 50  0000 L CNN
-F 2 "Resistors_SMD:R_0603" H 4500 3550 60  0001 C CNN
+F 2 "Resistor_SMD:R_0603_1608Metric" H 4500 3550 60  0001 C CNN
 F 3 "" H 4500 3550 60  0000 C CNN
 F 4 "RMCF0603JT10K0" H 100 0   50  0001 C CNN "MPN"
@@
 F 0 "C53" V 3950 3200 50  0000 L CNN
 F 1 "100nF" V 3800 3000 50  0000 L CNN
-F 2 "Capacitors_SMD:C_0603" H 3900 3150 60  0001 C CNN
+F 2 "Capacitor_SMD:C_0603_1608Metric" H 3900 3150 60  0001 C CNN
 F 3 "" H 3900 3150 60  0000 C CNN
 F 4 "C1608X7R1E104K080AA" H 100 0   50  0001 C CNN "MPN"

Commit message: correct tracks that overlap with new footprints
Changed lines of the file:
@@
 	4100 3450 4050 3450
 Wire Wire Line
-	4100 3100 4100 3450
+	4100 3100 4100 3150
 Wire Wire Line
 	4050 3750 4200 3750
@@
 	4100 3850 4100 3950
 Wire Wire Line
-	2950 3550 3450 3550
+	2950 3550 3150 3550
 Wire Wire Line
 	3150 3650 3150 3550
 Wire Wire Line
-	3250 3750 3250 4350
+	3250 3750 3250 3900
 Wire Wire Line
 	3250 3750 3450 3750
@@
 	7950 3200 7950 3250
 Wire Wire Line
-	7950 3450 7950 3650
+	7950 3450 7950 3550
 Wire Wire Line
 	7800 3550 7950 3550
@@
 	8500 3450 8500 3550
 Wire Wire Line
-	8500 3750 8500 3950
+	8500 3750 8500 3850
 Wire Wire Line
 	8500 4350 8500 4450
@@
 	9950 4700 9950 2750
 Wire Wire Line
-	4400 3750 4650 3750
+	4400 3750 4500 3750
 Wire Wire Line
 	8800 4150 8950 4150
@@
 NoConn ~ 2650 3350
 NoConn ~ 1850 3350
+Wire Wire Line
+	3150 3550 3450 3550
+Wire Wire Line
+	3250 3900 3250 4350
+Wire Wire Line
+	7950 3550 7950 3650
+Wire Wire Line
+	8500 3850 8500 3950
+Wire Wire Line
+	4500 3750 4650 3750
+Wire Wire Line
+	4100 3150 4100 3450
 $EndSCHEMATC
